File: INPUT/LB_BIT_i15_LIGHTTRIGGER/LB_BIT_i15_LIGHTTRIGGER-v02(rev1).brd (EAGLE design)
At the start: 20.3 x 32.1 mm, 51 parts

Commit message: Removed littlebits Logos in many of these
Parts:
- removed U$9: (no value), littleBits_Text:LB_V02
Changed lines of the file:
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@@
 <?xml version="1.0" encoding="utf-8"?>
 <!DOCTYPE eagle SYSTEM "eagle.dtd">
-<eagle version="6.1">
+<eagle version="6.2">
 <drawing>
 <settings>
@@
 <element name="I15BSF" library="bitSnap" package="BITSNAP_FEMALE" value="BITSNAP_FEMALE" x="1.27" y="0"/>
 <element name="U$8" library="ohw-logo" package="OSHW_FILLX150_NOTEXT" value="" x="8.4873" y="26.5719"/>
-<element name="U$9" library="littleBits_Text" package="LB_V02" value="" x="-0.635" y="3.4925"/>
 <element name="I15FD1" library="SparkFun" package="FIDUCIAL-1X2" value="FIDUCIAL1X2" x="1.905" y="5.08"/>
 <element name="I15FD2" library="SparkFun" package="FIDUCIAL-1X2" value="FIDUCIAL1X2" x="18.415" y="26.9875"/>
