File: INPUT/LB_BIT_i1-SLIDESWITCH/LB_BIT_i1_SLIDESWITCH-v03(rev2)/LB_BIT_i1_SLIDESWITCH-v03(rev2).brd (EAGLE design)
At the start: 21.4 x 25.5 mm, 9 parts

Commit message: Updated licenses
Parts:
- moved U$2 185.6 mm to (0.00, 0.00)
Changed lines of the file:
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@@
 <?xml version="1.0" encoding="utf-8"?>
 <!DOCTYPE eagle SYSTEM "eagle.dtd">
-<eagle version="6.1">
+<eagle version="6.6.0">
 <drawing>
 <settings>
@@
 <layer number="54" name="bGND_GNDA" color="1" fill="9" visible="no" active="no"/>
 <layer number="56" name="wert" color="7" fill="1" visible="yes" active="yes"/>
+<layer number="57" name="tCAD" color="7" fill="1" visible="no" active="no"/>
 <layer number="91" name="Nets" color="2" fill="1" visible="no" active="no"/>
 <layer number="92" name="Busses" color="1" fill="1" visible="no" active="no"/>
@@
 <layer number="145" name="DrillLegend_01-16" color="2" fill="9" visible="yes" active="yes"/>
 <layer number="146" name="DrillLegend_01-20" color="3" fill="9" visible="yes" active="yes"/>
+<layer number="150" name="Notes" color="7" fill="1" visible="yes" active="yes"/>
 <layer number="151" name="HeatSink" color="7" fill="1" visible="yes" active="yes"/>
 <layer number="152" name="_bDocu" color="7" fill="1" visible="yes" active="yes"/>
+<layer number="153" name="FabDoc1" color="6" fill="1" visible="no" active="no"/>
+<layer number="154" name="FabDoc2" color="2" fill="1" visible="no" active="no"/>
+<layer number="155" name="FabDoc3" color="7" fill="15" visible="no" active="no"/>
 <layer number="199" name="Contour" color="7" fill="1" visible="yes" active="yes"/>
 <layer number="200" name="200bmp" color="1" fill="10" visible="no" active="no"/>
@@
 <layer number="225" name="225bmp" color="26" fill="10" visible="yes" active="yes"/>
 <layer number="226" name="226bmp" color="27" fill="10" visible="yes" active="yes"/>
+<layer number="227" name="227bmp" color="7" fill="1" visible="yes" active="yes"/>
+<layer number="228" name="228bmp" color="7" fill="1" visible="yes" active="yes"/>
 <layer number="248" name="Housing" color="7" fill="1" visible="yes" active="yes"/>
 <layer number="249" name="Edge" color="7" fill="1" visible="yes" active="yes"/>
@@
 <wire x1="14.512" y1="22.992" x2="14.512" y2="24.008" width="0.1016" layer="146"/>
 <wire x1="14.512" y1="24.008" x2="15.02" y2="24.008" width="0.1016" layer="146"/>
-<dimension x1="3.8" y1="26.5" x2="16.6" y2="26.5" x3="10.2" y3="37.7" layer="47" dtype="horizontal"/>
-<dimension x1="20.4" y1="22" x2="0" y2="22" x3="10.2" y3="45.15" layer="47" dtype="horizontal"/>
-<dimension x1="-0.5" y1="4.5" x2="-0.5" y2="21.5" x3="-4.2" y3="13" layer="47" dtype="vertical"/>
-<dimension x1="3.3" y1="0" x2="3.3" y2="26" x3="-12.3" y3="13" layer="47" dtype="vertical"/>
+<dimension x1="3.8" y1="26.5" x2="16.6" y2="26.5" x3="10.2" y3="37.7" textsize="3.5" layer="47" dtype="horizontal"/>
+<dimension x1="20.4" y1="22" x2="0" y2="22" x3="10.2" y3="45.15" textsize="3.5" layer="47" dtype="horizontal"/>
+<dimension x1="-0.5" y1="4.5" x2="-0.5" y2="21.5" x3="-4.2" y3="13" textsize="3.5" layer="47" dtype="vertical"/>
+<dimension x1="3.3" y1="0" x2="3.3" y2="26" x3="-12.3" y3="13" textsize="3.5" layer="47" dtype="vertical"/>
 <text x="-5.95" y="52.9" size="1.778" layer="46">1mm DIA. ROUTER PATH</text>
-<dimension x1="4.35" y1="22" x2="16.05" y2="22" x3="10.2" y3="31.4" layer="47" dtype="horizontal"/>
+<dimension x1="4.35" y1="22" x2="16.05" y2="22" x3="10.2" y3="31.4" textsize="3.5" layer="47" dtype="horizontal"/>
 <text x="18.2" y="20.9" size="1.3" layer="21" font="vector" rot="SR270">i1 slide switch</text>
 <text x="4.7" y="9.4" size="1.3" layer="21" font="vector" rot="SR270">on</text>
@@
 </class>
 </classes>
-<designrules>
+<designrules name="default">
 <description language="en">&lt;b&gt;EAGLE Design Rules&lt;/b&gt;
 &lt;p&gt;
@@
 <element name="I1BSF1" library="bitSnap" package="BITSNAP_V03_FEMALE" value="BITSNAP_V03_FEMALE" x="3.75" y="0"/>
 <element name="I1BSM1" library="bitSnap" package="BITSNAP_V03_MALE" value="BITSNAP_V03_MALE" x="16.65" y="26" rot="R180"/>
-<element name="U$2" library="LITTLEBITS" package="FABDWG01-OHW" value="FRAME-LETTER-OHWOHW" x="-170.5" y="-73.4"/>
+<element name="U$2" library="LITTLEBITS" package="FABDWG01-OHW" value="FRAME-LETTER-OHWOHW" x="0" y="0"/>
 <element name="U$1" library="LITTLEBITS" package="OSHW-LOGO-L" value="OSHW-LOGOL" x="-39.4" y="-17.35"/>
 <element name="U$3" library="LITTLEBITS" package="OSHWCREDIT" value="LB_CREDITS" x="-6.5" y="-27.8"/>
@@
 </board>
 </drawing>
+<compatibility>
+<note version="6.3" minversion="6.2.2" severity="warning">
+Since Version 6.2.2 text objects can contain more than one line,
+which will not be processed correctly with this version.
+</note>
+</compatibility>
 </eagle>
