File: INPUT/LB_BIT_i11_PRESSURESENSOR/LB_i11_Pressure_Sensor-v03(4_4)/LB_i11_Pressure_Sensor-v03(4_4).brd (EAGLE design)
At the start: 21.4 x 11.5 mm, 16 parts

Commit message: Updated licenses
Parts:
- moved FRAME1 165.1 mm to (0.00, 0.00)
Changed lines of the file:
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@@
 <?xml version="1.0" encoding="utf-8"?>
 <!DOCTYPE eagle SYSTEM "eagle.dtd">
-<eagle version="6.1">
+<eagle version="6.6.0">
 <drawing>
 <settings>
@@
 <layer number="54" name="bGND_GNDA" color="1" fill="9" visible="no" active="no"/>
 <layer number="56" name="wert" color="7" fill="1" visible="yes" active="yes"/>
+<layer number="57" name="tCAD" color="7" fill="1" visible="no" active="no"/>
 <layer number="91" name="Nets" color="2" fill="1" visible="no" active="no"/>
 <layer number="92" name="Busses" color="1" fill="1" visible="no" active="no"/>
@@
 <layer number="145" name="DrillLegend_01-16" color="2" fill="9" visible="yes" active="yes"/>
 <layer number="146" name="DrillLegend_01-20" color="3" fill="9" visible="yes" active="yes"/>
+<layer number="150" name="Notes" color="7" fill="1" visible="yes" active="yes"/>
 <layer number="151" name="HeatSink" color="7" fill="1" visible="yes" active="yes"/>
 <layer number="152" name="_bDocu" color="7" fill="1" visible="yes" active="yes"/>
+<layer number="153" name="FabDoc1" color="6" fill="1" visible="no" active="no"/>
+<layer number="154" name="FabDoc2" color="2" fill="1" visible="no" active="no"/>
+<layer number="155" name="FabDoc3" color="7" fill="15" visible="no" active="no"/>
 <layer number="199" name="Contour" color="7" fill="1" visible="yes" active="yes"/>
 <layer number="200" name="200bmp" color="1" fill="10" visible="no" active="no"/>
@@
 <layer number="225" name="225bmp" color="26" fill="10" visible="yes" active="yes"/>
 <layer number="226" name="226bmp" color="27" fill="10" visible="yes" active="yes"/>
+<layer number="227" name="227bmp" color="7" fill="1" visible="yes" active="yes"/>
+<layer number="228" name="228bmp" color="7" fill="1" visible="yes" active="yes"/>
 <layer number="248" name="Housing" color="7" fill="1" visible="yes" active="yes"/>
 <layer number="249" name="Edge" color="7" fill="1" visible="yes" active="yes"/>
@@
 <wire x1="20.4" y1="15" x2="20.4" y2="4.5" width="0" layer="20"/>
 <text x="19.3" y="5.1" size="0.8128" layer="16" font="vector" ratio="12" rot="SMR90">rev4</text>
-<dimension x1="3.8" y1="20" x2="16.6" y2="20" x3="10.2" y3="31.2" layer="47" dtype="horizontal"/>
-<dimension x1="20.4" y1="15.5" x2="0" y2="15.5" x3="10.2" y3="38.65" layer="47" dtype="horizontal"/>
-<dimension x1="-0.5" y1="4.5" x2="-0.5" y2="15" x3="-4.2" y3="9.75" layer="47" dtype="vertical"/>
-<dimension x1="3.3" y1="0" x2="3.3" y2="19.5" x3="-12.3" y3="9.75" layer="47" dtype="vertical"/>
-<dimension x1="4.35" y1="15.5" x2="16.05" y2="15.5" x3="10.2" y3="24.9" layer="47" dtype="horizontal"/>
+<dimension x1="3.8" y1="20" x2="16.6" y2="20" x3="10.2" y3="31.2" textsize="3.5" layer="47" dtype="horizontal"/>
+<dimension x1="20.4" y1="15.5" x2="0" y2="15.5" x3="10.2" y3="38.65" textsize="3.5" layer="47" dtype="horizontal"/>
+<dimension x1="-0.5" y1="4.5" x2="-0.5" y2="15" x3="-4.2" y3="9.75" textsize="3.5" layer="47" dtype="vertical"/>
+<dimension x1="3.3" y1="0" x2="3.3" y2="19.5" x3="-12.3" y3="9.75" textsize="3.5" layer="47" dtype="vertical"/>
+<dimension x1="4.35" y1="15.5" x2="16.05" y2="15.5" x3="10.2" y3="24.9" textsize="3.5" layer="47" dtype="horizontal"/>
 <wire x1="0" y1="15.5" x2="-0.5" y2="15.5" width="1" layer="46"/>
 <wire x1="-0.5" y1="15.5" x2="-0.5" y2="4" width="1" layer="46"/>
@@
 </class>
 </classes>
-<designrules>
+<designrules name="default">
 <description language="de">&lt;b&gt;EAGLE Design Rules&lt;/b&gt;
 &lt;p&gt;
@@
 <attribute name="IEC_ESD_PROT0" value="+/-18kV" x="8.75" y="4.6" size="1.778" layer="28" rot="MR180" display="off"/>
 </element>
-<element name="FRAME1" library="LITTLEBITS" package="FABDWG01-OHW" value="FRAME-LETTER-OHWOHW" x="-146.4" y="-76.4"/>
+<element name="FRAME1" library="LITTLEBITS" package="FABDWG01-OHW" value="FRAME-LETTER-OHWOHW" x="0" y="0"/>
 <element name="U$1" library="LITTLEBITS" package="OSHW-LOGO-L" value="OSHW-LOGOL" x="-25.7" y="-70"/>
 </elements>
@@
 </board>
 </drawing>
+<compatibility>
+<note version="6.3" minversion="6.2.2" severity="warning">
+Since Version 6.2.2 text objects can contain more than one line,
+which will not be processed correctly with this version.
+</note>
+</compatibility>
 </eagle>

Commit message: Updated license text
Parts:
- moved U$7 18.5 mm to (-90.9, -62.8)
Changed lines of the file:
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@@
 </element>
 <element name="U$6" library="ohw-logo" package="OSHW_FILLX150_NOTEXT" value="" x="15.809" y="9.059"/>
-<element name="U$7" library="LITTLEBITS" package="OSHWCREDIT" value="LB_CREDITS" x="-72.88" y="-58.53"/>
+<element name="U$7" library="LITTLEBITS" package="OSHWCREDIT" value="LB_CREDITS" x="-90.93" y="-62.78"/>
 <element name="I11BSM1" library="bitSnap" package="BITSNAP_V03_MALE" value="BITSNAP_V03_MALE" x="16.65" y="19.5" rot="R180"/>
 <element name="I11BSF1" library="bitSnap" package="BITSNAP_V03_FEMALE" value="BITSNAP_V03_FEMALE" x="3.75" y="0"/>
