File: INPUT/LB_BIT_i13_LIGHTSENSOR/LB_BIT_i13_LIGHTSENSOR-v03(5_5)/LB_BIT_i13_LIGHTSENSOR-v03(5_5).brd (EAGLE design)
At the start: 21.4 x 18.1 mm, 38 parts

Commit message: Updated licenses
Parts:
- moved U$3 165.5 mm to (0.00, 0.00)
- moved U$1 107.7 mm to (-92.4, -65.2)
- moved U$2 48.5 mm to (-42.0, -60.6)
Changed lines of the file:
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@@
 <?xml version="1.0" encoding="utf-8"?>
 <!DOCTYPE eagle SYSTEM "eagle.dtd">
-<eagle version="6.1">
+<eagle version="6.6.0">
 <drawing>
 <settings>
@@
 <layer number="54" name="bGND_GNDA" color="7" fill="1" visible="no" active="no"/>
 <layer number="56" name="wert" color="7" fill="1" visible="no" active="no"/>
+<layer number="57" name="tCAD" color="7" fill="1" visible="no" active="no"/>
 <layer number="91" name="Nets" color="2" fill="1" visible="no" active="no"/>
 <layer number="92" name="Busses" color="1" fill="1" visible="no" active="no"/>
@@
 <layer number="145" name="DrillLegend_01-16" color="2" fill="9" visible="yes" active="yes"/>
 <layer number="146" name="DrillLegend_01-20" color="3" fill="9" visible="yes" active="yes"/>
+<layer number="150" name="Notes" color="7" fill="1" visible="yes" active="yes"/>
 <layer number="151" name="HeatSink" color="7" fill="1" visible="yes" active="yes"/>
 <layer number="152" name="_bDocu" color="7" fill="1" visible="yes" active="yes"/>
+<layer number="153" name="FabDoc1" color="6" fill="1" visible="no" active="no"/>
+<layer number="154" name="FabDoc2" color="2" fill="1" visible="no" active="no"/>
+<layer number="155" name="FabDoc3" color="7" fill="15" visible="no" active="no"/>
 <layer number="199" name="Contour" color="7" fill="1" visible="yes" active="yes"/>
 <layer number="200" name="200bmp" color="1" fill="10" visible="yes" active="yes"/>
@@
 <layer number="225" name="225bmp" color="26" fill="10" visible="yes" active="yes"/>
 <layer number="226" name="226bmp" color="27" fill="10" visible="yes" active="yes"/>
+<layer number="227" name="227bmp" color="7" fill="1" visible="yes" active="yes"/>
+<layer number="228" name="228bmp" color="7" fill="1" visible="yes" active="yes"/>
 <layer number="248" name="Housing" color="7" fill="1" visible="yes" active="yes"/>
 <layer number="249" name="Edge" color="7" fill="1" visible="yes" active="yes"/>
@@
 <text x="55.5" y="-44.7" size="1.3" layer="50">5</text>
 <text x="-11.35" y="-48.5" size="1.3" layer="50">LIGHT SENSOR BIT</text>
-<dimension x1="3.8" y1="27" x2="16.6" y2="27" x3="10.2" y3="33.5" layer="47" dtype="horizontal"/>
-<dimension x1="0" y1="22.5" x2="20.4" y2="22.5" x3="10.2" y3="37.65" layer="47" dtype="horizontal"/>
-<dimension x1="2.8" y1="26.1" x2="2.8" y2="0" x3="-10.45" y3="13.05" layer="47" dtype="vertical"/>
-<dimension x1="-1" y1="4.5" x2="-1" y2="21.5" x3="-5.4" y3="13" layer="47" dtype="vertical"/>
-<dimension x1="4.35" y1="22.5" x2="16.05" y2="22.5" x3="10.2" y3="29.25" layer="47" dtype="horizontal"/>
+<dimension x1="3.8" y1="27" x2="16.6" y2="27" x3="10.2" y3="33.5" textsize="3.5" layer="47" dtype="horizontal"/>
+<dimension x1="0" y1="22.5" x2="20.4" y2="22.5" x3="10.2" y3="37.65" textsize="3.5" layer="47" dtype="horizontal"/>
+<dimension x1="2.8" y1="26.1" x2="2.8" y2="0" x3="-10.45" y3="13.05" textsize="3.5" layer="47" dtype="vertical"/>
+<dimension x1="-1" y1="4.5" x2="-1" y2="21.5" x3="-5.4" y3="13" textsize="3.5" layer="47" dtype="vertical"/>
+<dimension x1="4.35" y1="22.5" x2="16.05" y2="22.5" x3="10.2" y3="29.25" textsize="3.5" layer="47" dtype="horizontal"/>
 <text x="4.55" y="10.3" size="0.4064" layer="25" font="vector">I13VR1</text>
 <text x="4.95" y="6.15" size="0.4064" layer="25" font="vector">100K</text>
@@
 </class>
 </classes>
-<designrules>
+<designrules name="default">
 <description language="de">&lt;b&gt;EAGLE Design Rules&lt;/b&gt;
 &lt;p&gt;
@@
 <attribute name="VALUE" x="16.916" y="10.278" size="0.4064" layer="27" rot="R180"/>
 </element>
-<element name="U$1" library="LITTLEBITS" package="OSHWCREDIT" value="OSHWCREDIT" x="7.9" y="-26.1"/>
-<element name="U$2" library="LITTLEBITS" package="OSHW-LOGO-L" value="OSHW-LOGOL" x="-19.6" y="-17.6"/>
+<element name="U$2" library="LITTLEBITS" package="OSHW-LOGO-L" value="OSHW-LOGOL" x="-42" y="-60.6"/>
 <element name="I13C4" library="LITTLEBITS" package="CAP-0603" value="0.1u" x="18" y="12" smashed="yes" rot="MR0">
 <attribute name="LB_PN" value="" x="18" y="12" size="1.778" layer="28" rot="MR0" display="off"/>
@@
 <attribute name="VALUE" x="16.316" y="19.357" size="0.4064" layer="28" font="vector" rot="MR0"/>
 </element>
-<element name="U$3" library="LITTLEBITS" package="FABDWG01-OHW" value="FRAME-LETTER-OHWOHW" x="-146.8" y="-76.4"/>
+<element name="U$1" library="LITTLEBITS" package="OSHWCREDIT" value="OSHWCREDIT" x="-92.4" y="-65.2"/>
+<element name="U$3" library="LITTLEBITS" package="FABDWG01-OHW" value="FRAME-LETTER-OHWOHW" x="0" y="0"/>
 </elements>
 <signals>
@@
 </board>
 </drawing>
+<compatibility>
+<note version="6.3" minversion="6.2.2" severity="warning">
+Since Version 6.2.2 text objects can contain more than one line,
+which will not be processed correctly with this version.
+</note>
+</compatibility>
 </eagle>

Commit message: Updated license text
Parts:
- moved U$2 11.7 mm to (-34.0, -69.2)
Changed lines of the file:
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@@
 <attribute name="LB_PN" value="?" x="7.7" y="21.5" size="1.778" layer="28" rot="MR270" display="off"/>
 <attribute name="V_OPERATION" value="5V" x="7.7" y="21.5" size="1.778" layer="28" rot="MR270" display="off"/>
-<attribute name="IEC_ESD_PROT" value="+/-18kV" x="7.7" y="21.5" size="1.778" layer="28" rot="MR270" display="off"/>
 <attribute name="V_CLAMP" value="?" x="7.7" y="21.5" size="1.778" layer="28" rot="MR270" display="off"/>
 <attribute name="NAME" x="7.884" y="25.389" size="0.4064" layer="26" rot="MR270"/>
 <attribute name="VALUE" x="8.897" y="25.466" size="0.4064" layer="28" rot="MR270"/>
+<attribute name="MPN" value="ESD9B5.0ST5G" x="7.7" y="21.5" size="1.778" layer="28" rot="MR270" display="off"/>
+<attribute name="IEC_ESD_PROT0" value="+/-18kV" x="7.7" y="21.5" size="1.778" layer="28" rot="MR270" display="off"/>
 </element>
 <element name="I13TVS2" library="LITTLEBITS" package="SOD-923" value="ESD9B5.0ST5G" x="9" y="4.5" smashed="yes" rot="MR180">
 <attribute name="LB_PN" value="?" x="9" y="4.5" size="1.778" layer="28" rot="MR180" display="off"/>
 <attribute name="V_OPERATION" value="5V" x="9" y="4.5" size="1.778" layer="28" rot="MR180" display="off"/>
-<attribute name="IEC_ESD_PROT" value="+/-18kV" x="9" y="4.5" size="1.778" layer="28" rot="MR180" display="off"/>
 <attribute name="V_CLAMP" value="?" x="9" y="4.5" size="1.778" layer="28" rot="MR180" display="off"/>
 <attribute name="NAME" x="7.911" y="3.834" size="0.4064" layer="26" rot="MR180"/>
 <attribute name="VALUE" x="6.334" y="3.297" size="0.4064" layer="28" rot="MR180"/>
+<attribute name="MPN" value="ESD9B5.0ST5G" x="9" y="4.5" size="1.778" layer="28" rot="MR180" display="off"/>
+<attribute name="IEC_ESD_PROT0" value="+/-18kV" x="9" y="4.5" size="1.778" layer="28" rot="MR180" display="off"/>
 </element>
 <element name="I13C2" library="LITTLEBITS" package="CAP-0603" value="0.1u" x="2.5" y="19.9" smashed="yes" rot="MR0">
@@
 <attribute name="VALUE" x="16.916" y="10.278" size="0.4064" layer="27" rot="R180"/>
 </element>
-<element name="U$2" library="LITTLEBITS" package="OSHW-LOGO-L" value="OSHW-LOGOL" x="-42" y="-60.6"/>
+<element name="U$2" library="LITTLEBITS" package="OSHW-LOGO-L" value="OSHW-LOGOL" x="-34" y="-69.2"/>
 <element name="I13C4" library="LITTLEBITS" package="CAP-0603" value="0.1u" x="18" y="12" smashed="yes" rot="MR0">
 <attribute name="LB_PN" value="" x="18" y="12" size="1.778" layer="28" rot="MR0" display="off"/>
