File: INPUT/LB_BIT_i16_PULSE/LB_i16-Pulse-v03(rev2)/LB_i16-Pulse-v03(rev2).sch (EAGLE design)
At the start: 17 parts

Commit message: Updated licenses
Parts:
- removed U$19: LB_CREDITS_V2, LITTLEBITS:LB_CREDITS_V2
- added U$1: OSHWCREDIT, LITTLEBITS:OSHWCREDIT
- renumbered U$18 to U$2
Changed lines of the file:
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@@
 <?xml version="1.0" encoding="utf-8"?>
 <!DOCTYPE eagle SYSTEM "eagle.dtd">
-<eagle version="6.1">
+<eagle version="6.6.0">
 <drawing>
 <settings>
@@
 <layer number="54" name="bGND_GNDA" color="1" fill="9" visible="no" active="no"/>
 <layer number="56" name="wert" color="7" fill="1" visible="no" active="no"/>
+<layer number="57" name="tCAD" color="7" fill="1" visible="no" active="no"/>
 <layer number="91" name="Nets" color="2" fill="1" visible="yes" active="yes"/>
 <layer number="92" name="Busses" color="1" fill="1" visible="yes" active="yes"/>
@@
 <layer number="145" name="DrillLegend_01-16" color="2" fill="9" visible="yes" active="yes"/>
 <layer number="146" name="DrillLegend_01-20" color="3" fill="9" visible="yes" active="yes"/>
+<layer number="150" name="Notes" color="7" fill="1" visible="yes" active="yes"/>
 <layer number="151" name="HeatSink" color="7" fill="1" visible="no" active="yes"/>
 <layer number="152" name="_bDocu" color="7" fill="1" visible="yes" active="yes"/>
+<layer number="153" name="FabDoc1" color="6" fill="1" visible="no" active="no"/>
+<layer number="154" name="FabDoc2" color="2" fill="1" visible="no" active="no"/>
+<layer number="155" name="FabDoc3" color="7" fill="15" visible="no" active="no"/>
 <layer number="199" name="Contour" color="7" fill="1" visible="yes" active="yes"/>
 <layer number="200" name="200bmp" color="1" fill="10" visible="no" active="yes"/>
@@
 <layer number="225" name="225bmp" color="26" fill="10" visible="no" active="yes"/>
 <layer number="226" name="226bmp" color="27" fill="10" visible="no" active="yes"/>
+<layer number="227" name="227bmp" color="7" fill="1" visible="yes" active="yes"/>
+<layer number="228" name="228bmp" color="7" fill="1" visible="yes" active="yes"/>
 <layer number="248" name="Housing" color="7" fill="1" visible="yes" active="yes"/>
 <layer number="249" name="Edge" color="7" fill="1" visible="yes" active="yes"/>
@@
 <part name="GND5" library="SparkFun" deviceset="GND" device=""/>
 <part name="U$3" library="SparkFun_NEW" deviceset="OSHW-LOGO" device="L"/>
-<part name="U$19" library="LITTLEBITS" deviceset="LB_CREDITS_V2" device=""/>
 <part name="I16BSM1" library="bitSnap" deviceset="BITSNAP_V03_MALE" device=""/>
 <part name="I16BSF1" library="bitSnap" deviceset="BITSNAP_V03_FEMALE" device=""/>
-<part name="U$18" library="LITTLEBITS" deviceset="FRAME-LETTER-OHW" device="OHW"/>
+<part name="U$1" library="LITTLEBITS" deviceset="OSHWCREDIT" device=""/>
+<part name="U$2" library="LITTLEBITS" deviceset="FRAME-LETTER-OHW" device="OHW"/>
 </parts>
 <sheets>
@@
 <instance part="GND5" gate="1" x="182.88" y="127"/>
 <instance part="U$3" gate="G$1" x="132.08" y="12.7"/>
-<instance part="U$19" gate="G$1" x="50.8" y="10.16"/>
 <instance part="I16BSM1" gate="G$1" x="58.42" y="93.98"/>
 <instance part="I16BSF1" gate="G$1" x="193.04" y="93.98"/>
-<instance part="U$18" gate="G$1" x="0" y="0"/>
-<instance part="U$18" gate="G$2" x="147.32" y="0"/>
+<instance part="U$1" gate="G$1" x="71.12" y="10.16"/>
+<instance part="U$2" gate="G$1" x="0" y="0"/>
+<instance part="U$2" gate="G$2" x="147.32" y="0"/>
 </instances>
 <busses>
@@
 </schematic>
 </drawing>
+<compatibility>
+<note version="6.3" minversion="6.2.2" severity="warning">
+Since Version 6.2.2 text objects can contain more than one line,
+which will not be processed correctly with this version.
+</note>
+</compatibility>
 </eagle>

Commit message: Updated license text
Parts:
- I16U3: value LV321SOT-235 -> LV321SOT23-5; device LITTLEBITS:LV321SOT-235 -> LITTLEBITS:LV321SOT23-5
Changed lines of the file:
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@@
 <part name="I16C1" library="SparkFun" deviceset="CAP" device="0603-CAP" value="0.1uF"/>
 <part name="I16C3" library="SparkFun" deviceset="CAP" device="0603-CAP" value="0.1uF"/>
-<part name="I16U3" library="LITTLEBITS" deviceset="LV321" device="SOT-235"/>
+<part name="I16U3" library="LITTLEBITS" deviceset="LV321" device="SOT23-5"/>
 <part name="GND3" library="SparkFun" deviceset="GND" device=""/>
 <part name="P+3" library="SparkFun" deviceset="VCC" device=""/>
@@
 <instance part="I16BSM1" gate="G$1" x="58.42" y="93.98"/>
 <instance part="I16BSF1" gate="G$1" x="193.04" y="93.98"/>
-<instance part="U$1" gate="G$1" x="71.12" y="10.16"/>
+<instance part="U$1" gate="G$1" x="48.26" y="10.16"/>
 <instance part="U$2" gate="G$1" x="0" y="0"/>
 <instance part="U$2" gate="G$2" x="147.32" y="0"/>
