File: INPUT/LB_BIT_i17_TIMEOUT/LB_BIT_i17_TIMEOUT-v03(rev1)/LB_BIT_i17_timeout-v03(rev1).brd (EAGLE design)
At the start: 21.4 x 18.1 mm, 23 parts

Commit message: Updated licenses
Parts:
- removed FRAME1: FRAME-LETTER-OHWOHW, LITTLEBITS:FABDWG01-OHW
- removed U$20: LB_CREDITS_V2, LITTLEBITS:LB_CREDITS_V2
- added U$1: OSHWCREDIT, LITTLEBITS:OSHWCREDIT
- added U$2: FRAME-LETTER-OHWOHW, LITTLEBITS:FABDWG01-OHW
- moved U$4 44.5 mm to (113.8, 16.9)
Changed lines of the file:
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@@
 <?xml version="1.0" encoding="utf-8"?>
 <!DOCTYPE eagle SYSTEM "eagle.dtd">
-<eagle version="6.1">
+<eagle version="6.6.0">
 <drawing>
 <settings>
@@
 <layer number="54" name="bGND_GNDA" color="1" fill="9" visible="no" active="no"/>
 <layer number="56" name="wert" color="7" fill="1" visible="yes" active="yes"/>
+<layer number="57" name="tCAD" color="7" fill="1" visible="no" active="no"/>
 <layer number="91" name="Nets" color="2" fill="1" visible="no" active="no"/>
 <layer number="92" name="Busses" color="1" fill="1" visible="no" active="no"/>
@@
 <layer number="145" name="DrillLegend_01-16" color="2" fill="9" visible="yes" active="yes"/>
 <layer number="146" name="DrillLegend_01-20" color="3" fill="9" visible="yes" active="yes"/>
+<layer number="150" name="Notes" color="7" fill="1" visible="yes" active="yes"/>
 <layer number="151" name="HeatSink" color="7" fill="1" visible="yes" active="yes"/>
 <layer number="152" name="_bDocu" color="7" fill="1" visible="yes" active="yes"/>
+<layer number="153" name="FabDoc1" color="6" fill="1" visible="no" active="no"/>
+<layer number="154" name="FabDoc2" color="2" fill="1" visible="no" active="no"/>
+<layer number="155" name="FabDoc3" color="7" fill="15" visible="no" active="no"/>
 <layer number="199" name="Contour" color="7" fill="1" visible="yes" active="yes"/>
 <layer number="200" name="200bmp" color="1" fill="10" visible="no" active="no"/>
@@
 <layer number="225" name="225bmp" color="26" fill="10" visible="yes" active="yes"/>
 <layer number="226" name="226bmp" color="27" fill="10" visible="yes" active="yes"/>
+<layer number="227" name="227bmp" color="7" fill="1" visible="yes" active="yes"/>
+<layer number="228" name="228bmp" color="7" fill="1" visible="yes" active="yes"/>
 <layer number="248" name="Housing" color="7" fill="1" visible="yes" active="yes"/>
 <layer number="249" name="Edge" color="7" fill="1" visible="yes" active="yes"/>
@@
 <wire x1="184.94" y1="97.2" x2="184.94" y2="79.1" width="1" layer="46"/>
 <wire x1="163.54" y1="79.1" x2="163.54" y2="97.2" width="1" layer="46"/>
-<dimension x1="167.84" y1="101.6" x2="180.64" y2="101.6" x3="174.24" y3="112.8" layer="47" dtype="horizontal"/>
-<dimension x1="184.44" y1="97.1" x2="164.04" y2="97.1" x3="174.24" y3="120" layer="47" dtype="horizontal"/>
-<dimension x1="163.54" y1="79.6" x2="163.54" y2="96.6" x3="159.84" y3="88.1" layer="47" dtype="vertical"/>
-<dimension x1="167.34" y1="75.1" x2="167.34" y2="101.1" x3="151.74" y3="88.1" layer="47" dtype="vertical"/>
-<dimension x1="168.39" y1="97.2" x2="180.09" y2="97.2" x3="174.24" y3="106.7" layer="47" dtype="horizontal"/>
+<dimension x1="167.84" y1="101.6" x2="180.64" y2="101.6" x3="174.24" y3="112.8" textsize="3.5" layer="47" dtype="horizontal"/>
+<dimension x1="184.44" y1="97.1" x2="164.04" y2="97.1" x3="174.24" y3="120" textsize="3.5" layer="47" dtype="horizontal"/>
+<dimension x1="163.54" y1="79.6" x2="163.54" y2="96.6" x3="159.84" y3="88.1" textsize="3.5" layer="47" dtype="vertical"/>
+<dimension x1="167.34" y1="75.1" x2="167.34" y2="101.1" x3="151.74" y3="88.1" textsize="3.5" layer="47" dtype="vertical"/>
+<dimension x1="168.39" y1="97.2" x2="180.09" y2="97.2" x3="174.24" y3="106.7" textsize="3.5" layer="47" dtype="horizontal"/>
 <wire x1="176.04" y1="83.958" x2="176.04" y2="82.942" width="0.1016" layer="145"/>
 <wire x1="175.532" y1="83.45" x2="176.548" y2="83.45" width="0.1016" layer="145"/>
@@
 </class>
 </classes>
-<designrules>
+<designrules name="default">
 <description language="en">&lt;b&gt;EAGLE Design Rules&lt;/b&gt;
 &lt;p&gt;
@@
 <attribute name="VALUE" x="180.208159375" y="90.9515" size="0.4064" layer="28" font="vector" rot="MR90"/>
 </element>
-<element name="U$20" library="LITTLEBITS" package="LB_CREDITS_V2" value="LB_CREDITS_V2" x="163.015" y="46.42"/>
-<element name="U$4" library="SparkFun_NEW" package="OSHW-LOGO-L" value="OSHW-LOGOL" x="144.2375" y="49.33"/>
+<element name="U$4" library="SparkFun_NEW" package="OSHW-LOGO-L" value="OSHW-LOGOL" x="113.8375" y="16.88"/>
 <element name="I17BSM1" library="bitSnap" package="BITSNAP_V03_MALE" value="BITSNAP_V03_MALE" x="180.69" y="101.2" rot="R180"/>
 <element name="I17BSF1" library="bitSnap" package="BITSNAP_V03_FEMALE" value="BITSNAP_V03_FEMALE" x="167.79" y="75.1"/>
-<element name="FRAME1" library="LITTLEBITS" package="FABDWG01-OHW" value="FRAME-LETTER-OHWOHW" x="0" y="0" locked="yes"/>
+<element name="U$1" library="LITTLEBITS" package="OSHWCREDIT" value="OSHWCREDIT" x="51.95" y="12.1"/>
+<element name="U$2" library="LITTLEBITS" package="FABDWG01-OHW" value="FRAME-LETTER-OHWOHW" x="145.4" y="75.75"/>
 </elements>
 <signals>
@@
 </board>
 </drawing>
+<compatibility>
+<note version="6.3" minversion="6.2.2" severity="warning">
+Since Version 6.2.2 text objects can contain more than one line,
+which will not be processed correctly with this version.
+</note>
+</compatibility>
 </eagle>

Commit message: Updated license text
Parts:
- moved U$4 8.42 mm to (110.4, 9.18)
- moved U$1 1.66 mm to (51.2, 13.6)
Changed lines of the file:
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@@
 <attribute name="VALUE" x="180.208159375" y="90.9515" size="0.4064" layer="28" font="vector" rot="MR90"/>
 </element>
-<element name="U$4" library="SparkFun_NEW" package="OSHW-LOGO-L" value="OSHW-LOGOL" x="113.8375" y="16.88"/>
+<element name="U$4" library="SparkFun_NEW" package="OSHW-LOGO-L" value="OSHW-LOGOL" x="110.4375" y="9.18"/>
 <element name="I17BSM1" library="bitSnap" package="BITSNAP_V03_MALE" value="BITSNAP_V03_MALE" x="180.69" y="101.2" rot="R180"/>
 <element name="I17BSF1" library="bitSnap" package="BITSNAP_V03_FEMALE" value="BITSNAP_V03_FEMALE" x="167.79" y="75.1"/>
-<element name="U$1" library="LITTLEBITS" package="OSHWCREDIT" value="OSHWCREDIT" x="51.95" y="12.1"/>
 <element name="U$2" library="LITTLEBITS" package="FABDWG01-OHW" value="FRAME-LETTER-OHWOHW" x="145.4" y="75.75"/>
+<element name="U$1" library="LITTLEBITS" package="OSHWCREDIT" value="OSHWCREDIT" x="51.25" y="13.6"/>
 </elements>
 <signals>
