File: INPUT/LB_BIT_i19_ROLLERSWITCH/LB_BIT_i19_ROLLERSWITCH-v03(rev3)/LB_BIT_i19_ROLLERSWITCH-v03(rev3).brd (EAGLE design)
At the start: 21.4 x 24.7 mm, 10 parts

Commit message: Updated licenses
Parts:
- moved FRAME1 180.4 mm to (0.00, 0.00)
- moved U$1 110.1 mm to (-93.5, -63.6)
- moved U$3 48.1 mm to (-37.5, -59.0)
Changed lines of the file:
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@@
 <?xml version="1.0" encoding="utf-8"?>
 <!DOCTYPE eagle SYSTEM "eagle.dtd">
-<eagle version="6.1">
+<eagle version="6.6.0">
 <drawing>
 <settings>
@@
 <layer number="54" name="bGND_GNDA" color="1" fill="9" visible="no" active="no"/>
 <layer number="56" name="wert" color="7" fill="1" visible="yes" active="yes"/>
+<layer number="57" name="tCAD" color="7" fill="1" visible="no" active="no"/>
 <layer number="91" name="Nets" color="2" fill="1" visible="no" active="no"/>
 <layer number="92" name="Busses" color="1" fill="1" visible="no" active="no"/>
@@
 <layer number="145" name="DrillLegend_01-16" color="2" fill="9" visible="yes" active="yes"/>
 <layer number="146" name="DrillLegend_01-20" color="3" fill="9" visible="yes" active="yes"/>
+<layer number="150" name="Notes" color="7" fill="1" visible="yes" active="yes"/>
 <layer number="151" name="HeatSink" color="7" fill="1" visible="yes" active="yes"/>
 <layer number="152" name="_bDocu" color="7" fill="1" visible="yes" active="yes"/>
+<layer number="153" name="FabDoc1" color="6" fill="1" visible="no" active="no"/>
+<layer number="154" name="FabDoc2" color="2" fill="1" visible="no" active="no"/>
+<layer number="155" name="FabDoc3" color="7" fill="15" visible="no" active="no"/>
 <layer number="199" name="Contour" color="7" fill="1" visible="yes" active="yes"/>
 <layer number="200" name="200bmp" color="1" fill="10" visible="no" active="no"/>
@@
 <layer number="225" name="225bmp" color="26" fill="10" visible="yes" active="yes"/>
 <layer number="226" name="226bmp" color="27" fill="10" visible="yes" active="yes"/>
+<layer number="227" name="227bmp" color="7" fill="1" visible="yes" active="yes"/>
+<layer number="228" name="228bmp" color="7" fill="1" visible="yes" active="yes"/>
 <layer number="248" name="Housing" color="7" fill="1" visible="yes" active="yes"/>
 <layer number="249" name="Edge" color="7" fill="1" visible="yes" active="yes"/>
@@
 <wire x1="20.9" y1="28.7" x2="20.9" y2="4" width="1" layer="46"/>
 <wire x1="-0.5" y1="4" x2="-0.5" y2="28.7" width="1" layer="46"/>
-<dimension x1="3.8" y1="33.2" x2="16.6" y2="33.2" x3="10.2" y3="44.4" layer="47" dtype="horizontal"/>
-<dimension x1="20.4" y1="28.7" x2="0" y2="28.7" x3="10.2" y3="51.85" layer="47" dtype="horizontal"/>
-<dimension x1="-0.5" y1="4.5" x2="-0.5" y2="28.2" x3="-4.2" y3="16.35" layer="47" dtype="vertical"/>
-<dimension x1="3.3" y1="0" x2="3.3" y2="32.7" x3="-12.3" y3="16.35" layer="47" dtype="vertical"/>
-<dimension x1="4.35" y1="28.7" x2="16.05" y2="28.7" x3="10.2" y3="38.1" layer="47" dtype="horizontal"/>
+<dimension x1="3.8" y1="33.2" x2="16.6" y2="33.2" x3="10.2" y3="44.4" textsize="3.5" layer="47" dtype="horizontal"/>
+<dimension x1="20.4" y1="28.7" x2="0" y2="28.7" x3="10.2" y3="51.85" textsize="3.5" layer="47" dtype="horizontal"/>
+<dimension x1="-0.5" y1="4.5" x2="-0.5" y2="28.2" x3="-4.2" y3="16.35" textsize="3.5" layer="47" dtype="vertical"/>
+<dimension x1="3.3" y1="0" x2="3.3" y2="32.7" x3="-12.3" y3="16.35" textsize="3.5" layer="47" dtype="vertical"/>
+<dimension x1="4.35" y1="28.7" x2="16.05" y2="28.7" x3="10.2" y3="38.1" textsize="3.5" layer="47" dtype="horizontal"/>
 <text x="0.8" y="23.15" size="1.016" layer="25">I19SW2</text>
 <text x="-5.75" y="-20" size="1.778" layer="46">1mm DIA. ROUTER PATH</text>
@@
 </class>
 </classes>
-<designrules>
+<designrules name="default">
 <description language="en">&lt;b&gt;EAGLE Design Rules&lt;/b&gt;
 &lt;p&gt;
@@
 <element name="I19SW2" library="LITTLEBITS" package="ROLLERSWITCH-OMRON-D2F-01FL-A" value="ROLLERSWITCH-OMRON-SS-5GL2DRIGHTANGLE" x="6.6" y="9.8875" rot="R90"/>
 <element name="U$20" library="ohw-logo" package="OSHW_FILLX150_NOTEXT" value="" x="15.799" y="22.434"/>
-<element name="U$3" library="SparkFun_NEW" package="OSHW-LOGO-L" value="OSHW-LOGOL" x="-19.92" y="-14.23"/>
+<element name="U$3" library="SparkFun_NEW" package="OSHW-LOGO-L" value="OSHW-LOGOL" x="-37.52" y="-59.03"/>
 <element name="I19BSF1" library="bitSnap" package="BITSNAP_V03_FEMALE" value="BITSNAP_V03_FEMALE" x="3.75" y="0"/>
 <element name="I19BSM1" library="bitSnap" package="BITSNAP_V03_MALE" value="BITSNAP_V03_MALE" x="16.65" y="32.7" rot="R180"/>
-<element name="FRAME1" library="LITTLEBITS" package="FABDWG01-OHW" value="FRAME-LETTER-OHWOHW" x="-165.9" y="-70.95"/>
-<element name="U$1" library="LITTLEBITS" package="OSHWCREDIT" value="OSHWCREDIT" x="8.9" y="-23.2"/>
+<element name="FRAME1" library="LITTLEBITS" package="FABDWG01-OHW" value="FRAME-LETTER-OHWOHW" x="0" y="0"/>
+<element name="U$1" library="LITTLEBITS" package="OSHWCREDIT" value="OSHWCREDIT" x="-93.5" y="-63.6"/>
 </elements>
 <signals>
@@
 </board>
 </drawing>
+<compatibility>
+<note version="6.3" minversion="6.2.2" severity="warning">
+Since Version 6.2.2 text objects can contain more than one line,
+which will not be processed correctly with this version.
+</note>
+</compatibility>
 </eagle>

Commit message: Updated license text
Parts:
- moved U$3 10.8 mm to (-33.6, -69.1)
Changed lines of the file:
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@@
 <element name="I19SW2" library="LITTLEBITS" package="ROLLERSWITCH-OMRON-D2F-01FL-A" value="ROLLERSWITCH-OMRON-SS-5GL2DRIGHTANGLE" x="6.6" y="9.8875" rot="R90"/>
 <element name="U$20" library="ohw-logo" package="OSHW_FILLX150_NOTEXT" value="" x="15.799" y="22.434"/>
-<element name="U$3" library="SparkFun_NEW" package="OSHW-LOGO-L" value="OSHW-LOGOL" x="-37.52" y="-59.03"/>
+<element name="U$3" library="SparkFun_NEW" package="OSHW-LOGO-L" value="OSHW-LOGOL" x="-33.57" y="-69.13"/>
 <element name="I19BSF1" library="bitSnap" package="BITSNAP_V03_FEMALE" value="BITSNAP_V03_FEMALE" x="3.75" y="0"/>
 <element name="I19BSM1" library="bitSnap" package="BITSNAP_V03_MALE" value="BITSNAP_V03_MALE" x="16.65" y="32.7" rot="R180"/>
