File: INPUT/LB_BIT_i20_SOUNDTRIGGER/LB_BIT_i20_SOUNDTRIGGER-v03(rev1)/LB_BIT_i20_SOUNDTRIGGER-v03(rev1).brd (EAGLE design)
At the start: 21.4 x 18.1 mm, 32 parts

Commit message: Updated licenses
Parts:
- removed FRAME1: FRAME-LETTER-OHWOHW, LITTLEBITS:FABDWG01-OHW
- removed U$28: LB_CREDITS_V2, LITTLEBITS:LB_CREDITS_V2
- added U$1: OSHWCREDIT, LITTLEBITS:OSHWCREDIT
- added U$5: FRAME-LETTER-OHWOHW, LITTLEBITS:FABDWG01-OHW
- moved U$29 63.7 mm to (-37.2, -59.3)
Changed lines of the file:
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@@
 <?xml version="1.0" encoding="utf-8"?>
 <!DOCTYPE eagle SYSTEM "eagle.dtd">
-<eagle version="6.1">
+<eagle version="6.6.0">
 <drawing>
 <settings>
@@
 <layer number="54" name="bGND_GNDA" color="1" fill="9" visible="yes" active="yes"/>
 <layer number="56" name="wert" color="7" fill="1" visible="yes" active="yes"/>
+<layer number="57" name="tCAD" color="7" fill="1" visible="no" active="no"/>
 <layer number="91" name="Nets" color="2" fill="1" visible="no" active="no"/>
 <layer number="92" name="Busses" color="1" fill="1" visible="no" active="no"/>
@@
 <layer number="145" name="DrillLegend_01-16" color="2" fill="9" visible="yes" active="yes"/>
 <layer number="146" name="DrillLegend_01-20" color="3" fill="9" visible="yes" active="yes"/>
+<layer number="150" name="Notes" color="7" fill="1" visible="yes" active="yes"/>
 <layer number="151" name="HeatSink" color="7" fill="1" visible="yes" active="yes"/>
 <layer number="152" name="_bDocu" color="7" fill="1" visible="yes" active="yes"/>
+<layer number="153" name="FabDoc1" color="6" fill="1" visible="no" active="no"/>
+<layer number="154" name="FabDoc2" color="2" fill="1" visible="no" active="no"/>
+<layer number="155" name="FabDoc3" color="7" fill="15" visible="no" active="no"/>
 <layer number="199" name="Contour" color="7" fill="1" visible="yes" active="yes"/>
 <layer number="200" name="200bmp" color="1" fill="10" visible="yes" active="yes"/>
@@
 <layer number="225" name="225bmp" color="26" fill="10" visible="yes" active="yes"/>
 <layer number="226" name="226bmp" color="27" fill="10" visible="yes" active="yes"/>
+<layer number="227" name="227bmp" color="7" fill="1" visible="yes" active="yes"/>
+<layer number="228" name="228bmp" color="7" fill="1" visible="yes" active="yes"/>
 <layer number="248" name="Housing" color="7" fill="1" visible="yes" active="yes"/>
 <layer number="249" name="Edge" color="7" fill="1" visible="yes" active="yes"/>
@@
 <wire x1="20.9" y1="22.1" x2="20.9" y2="4" width="1" layer="46"/>
 <wire x1="-0.5" y1="4" x2="-0.5" y2="22.1" width="1" layer="46"/>
-<dimension x1="3.8" y1="26.6" x2="16.6" y2="26.6" x3="10.2" y3="37.8" layer="47" dtype="horizontal"/>
-<dimension x1="20.4" y1="22.1" x2="0" y2="22.1" x3="10.2" y3="45.25" layer="47" dtype="horizontal"/>
-<dimension x1="-0.5" y1="4.6" x2="-0.5" y2="21.6" x3="-4.2" y3="13.1" layer="47" dtype="vertical"/>
-<dimension x1="3.3" y1="0.1" x2="3.3" y2="26.1" x3="-12.3" y3="13.1" layer="47" dtype="vertical"/>
-<dimension x1="4.35" y1="22.1" x2="16.05" y2="22.1" x3="10.2" y3="31.5" layer="47" dtype="horizontal"/>
+<dimension x1="3.8" y1="26.6" x2="16.6" y2="26.6" x3="10.2" y3="37.8" textsize="3.5" layer="47" dtype="horizontal"/>
+<dimension x1="20.4" y1="22.1" x2="0" y2="22.1" x3="10.2" y3="45.25" textsize="3.5" layer="47" dtype="horizontal"/>
+<dimension x1="-0.5" y1="4.6" x2="-0.5" y2="21.6" x3="-4.2" y3="13.1" textsize="3.5" layer="47" dtype="vertical"/>
+<dimension x1="3.3" y1="0.1" x2="3.3" y2="26.1" x3="-12.3" y3="13.1" textsize="3.5" layer="47" dtype="vertical"/>
+<dimension x1="4.35" y1="22.1" x2="16.05" y2="22.1" x3="10.2" y3="31.5" textsize="3.5" layer="47" dtype="horizontal"/>
 <wire x1="12.6" y1="21.258" x2="12.6" y2="20.242" width="0.1016" layer="145"/>
 <wire x1="12.092" y1="20.75" x2="13.108" y2="20.75" width="0.1016" layer="145"/>
@@
 <wire x1="14.512" y1="23.6" x2="15.02" y2="24.108" width="0.1016" layer="146"/>
 <text x="-4.6" y="-11" size="1.778" layer="46">1mm DIA. ROUTER PATH</text>
-<text x="46.15" y="-53.15" size="1.778" layer="50">LB-BIT-i20-SOUNDTRIGGER-v03-GERBER-rev1 (8-31-2012)</text>
-<text x="40.65" y="-41.85" size="1.778" layer="50">i20 SOUND TRIGGER BIT PCB</text>
+<text x="-3.95" y="-59.2" size="1.778" layer="50">LB-BIT-i20-SOUNDTRIGGER-v03-GERBER-rev1 (8-31-2012)</text>
+<text x="-10.7" y="-48.15" size="1.778" layer="50">i20 SOUND TRIGGER BIT PCB</text>
 <text x="106.5" y="-37.75" size="1.778" layer="50">1</text>
 <text x="18.1" y="14.6" size="1.5" layer="21" font="vector" rot="SR270">i20</text>
@@
 </class>
 </classes>
-<designrules>
+<designrules name="default">
 <description language="en">&lt;b&gt;EAGLE Design Rules&lt;/b&gt;
 &lt;p&gt;
@@
 <attribute name="VALUE" x="12.474" y="8.962" size="0.4064" layer="28" rot="MR180"/>
 </element>
-<element name="U$28" library="LITTLEBITS" package="LB_CREDITS_V2" value="LB_CREDITS_V2" x="-16.65" y="-64.4"/>
-<element name="U$29" library="SparkFun_NEW" package="OSHW-LOGO-L" value="OSHW-LOGOL" x="26.25" y="-65.36"/>
+<element name="U$29" library="SparkFun_NEW" package="OSHW-LOGO-L" value="OSHW-LOGOL" x="-37.2" y="-59.31"/>
 <element name="I20Q1" library="transistor-small-signal" package="SOT363_PHILIPS" value="BC847BS" x="17.51" y="11.605" smashed="yes" rot="MR0">
 <attribute name="NAME" x="18.61" y="13.055" size="0.6096" layer="26" rot="MR0"/>
@@
 <element name="I20BSF1" library="bitSnap" package="BITSNAP_V03_FEMALE" value="BITSNAP_V03_FEMALE" x="3.75" y="0"/>
 <element name="I20BSM1" library="bitSnap" package="BITSNAP_V03_MALE" value="BITSNAP_V03_MALE" x="16.65" y="26.1" rot="R180"/>
-<element name="FRAME1" library="LITTLEBITS" package="FABDWG01-OHW" value="FRAME-LETTER-OHWOHW" x="-96.402665625" y="-69.55"/>
+<element name="U$1" library="LITTLEBITS" package="OSHWCREDIT" value="OSHWCREDIT" x="-92.85" y="-65.1"/>
+<element name="U$5" library="LITTLEBITS" package="FABDWG01-OHW" value="FRAME-LETTER-OHWOHW" x="0" y="0"/>
 </elements>
 <signals>
@@
 </board>
 </drawing>
+<compatibility>
+<note version="6.3" minversion="6.2.2" severity="warning">
+Since Version 6.2.2 text objects can contain more than one line,
+which will not be processed correctly with this version.
+</note>
+</compatibility>
 </eagle>

Commit message: Updated license text
Parts:
- moved U$29 8.36 mm to (-35.0, -67.4)
- moved U$1 3.00 mm to (-93.4, -62.1)
Changed lines of the file:
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@@
 <attribute name="VALUE" x="12.474" y="8.962" size="0.4064" layer="28" rot="MR180"/>
 </element>
-<element name="U$29" library="SparkFun_NEW" package="OSHW-LOGO-L" value="OSHW-LOGOL" x="-37.2" y="-59.31"/>
+<element name="U$29" library="SparkFun_NEW" package="OSHW-LOGO-L" value="OSHW-LOGOL" x="-34.95" y="-67.36"/>
 <element name="I20Q1" library="transistor-small-signal" package="SOT363_PHILIPS" value="BC847BS" x="17.51" y="11.605" smashed="yes" rot="MR0">
 <attribute name="NAME" x="18.61" y="13.055" size="0.6096" layer="26" rot="MR0"/>
@@
 <element name="I20BSF1" library="bitSnap" package="BITSNAP_V03_FEMALE" value="BITSNAP_V03_FEMALE" x="3.75" y="0"/>
 <element name="I20BSM1" library="bitSnap" package="BITSNAP_V03_MALE" value="BITSNAP_V03_MALE" x="16.65" y="26.1" rot="R180"/>
-<element name="U$1" library="LITTLEBITS" package="OSHWCREDIT" value="OSHWCREDIT" x="-92.85" y="-65.1"/>
 <element name="U$5" library="LITTLEBITS" package="FABDWG01-OHW" value="FRAME-LETTER-OHWOHW" x="0" y="0"/>
+<element name="U$1" library="LITTLEBITS" package="OSHWCREDIT" value="OSHWCREDIT" x="-93.4" y="-62.15"/>
 </elements>
 <signals>
