File: INPUT/LB_BIT_i20_SOUNDTRIGGER/LB_BIT_i20_SOUNDTRIGGER-v03(rev1)/LB_BIT_i20_SOUNDTRIGGER-v03(rev1).sch (EAGLE design)
At the start: 29 parts

Commit message: Updated licenses
Parts:
- removed U$28: LB_CREDITS_V2, LITTLEBITS:LB_CREDITS_V2
- added U$1: OSHWCREDIT, LITTLEBITS:OSHWCREDIT
- renumbered FRAME1 to U$5
Changed lines of the file:
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@@
 <?xml version="1.0" encoding="utf-8"?>
 <!DOCTYPE eagle SYSTEM "eagle.dtd">
-<eagle version="6.1">
+<eagle version="6.6.0">
 <drawing>
 <settings>
@@
 <layer number="54" name="bGND_GNDA" color="1" fill="9" visible="no" active="no"/>
 <layer number="56" name="wert" color="7" fill="1" visible="no" active="no"/>
+<layer number="57" name="tCAD" color="7" fill="1" visible="no" active="no"/>
 <layer number="91" name="Nets" color="2" fill="1" visible="yes" active="yes"/>
 <layer number="92" name="Busses" color="1" fill="1" visible="yes" active="yes"/>
@@
 <layer number="145" name="DrillLegend_01-16" color="2" fill="9" visible="yes" active="yes"/>
 <layer number="146" name="DrillLegend_01-20" color="3" fill="9" visible="yes" active="yes"/>
+<layer number="150" name="Notes" color="7" fill="1" visible="yes" active="yes"/>
 <layer number="151" name="HeatSink" color="7" fill="1" visible="yes" active="yes"/>
 <layer number="152" name="_bDocu" color="7" fill="1" visible="yes" active="yes"/>
+<layer number="153" name="FabDoc1" color="6" fill="1" visible="no" active="no"/>
+<layer number="154" name="FabDoc2" color="2" fill="1" visible="no" active="no"/>
+<layer number="155" name="FabDoc3" color="7" fill="15" visible="no" active="no"/>
 <layer number="199" name="Contour" color="7" fill="1" visible="yes" active="yes"/>
 <layer number="200" name="200bmp" color="1" fill="10" visible="no" active="no"/>
@@
 <layer number="225" name="225bmp" color="26" fill="10" visible="no" active="yes"/>
 <layer number="226" name="226bmp" color="27" fill="10" visible="no" active="yes"/>
+<layer number="227" name="227bmp" color="7" fill="1" visible="yes" active="yes"/>
+<layer number="228" name="228bmp" color="7" fill="1" visible="yes" active="yes"/>
 <layer number="248" name="Housing" color="7" fill="1" visible="yes" active="yes"/>
 <layer number="249" name="Edge" color="7" fill="1" visible="yes" active="yes"/>
@@
 <part name="I20U3" library="LITTLEBITS" deviceset="LV321" device="SOT23-5"/>
 <part name="I20P1" library="LITTLEBITS" deviceset="POT-TRIM-SMD-BOURNS-3303" device="" value="500K"/>
-<part name="FRAME1" library="LITTLEBITS" deviceset="FRAME-LETTER-OHW" device="OHW"/>
 <part name="I20R1" library="SparkFun" deviceset="RESISTOR" device="0603-RES" value="10K"/>
 <part name="I20R2" library="SparkFun" deviceset="RESISTOR" device="0603-RES" value="10K"/>
@@
 <part name="P+11" library="SparkFun" deviceset="VCC" device=""/>
 <part name="I20C6" library="SparkFun" deviceset="CAP" device="0805" value="10uF"/>
-<part name="U$28" library="LITTLEBITS" deviceset="LB_CREDITS_V2" device=""/>
 <part name="U$29" library="SparkFun_NEW" deviceset="OSHW-LOGO" device="L"/>
 <part name="I20Q1" library="transistor-small-signal" deviceset="BC847BS" device=""/>
@@
 <part name="I20BSF1" library="bitSnap" deviceset="BITSNAP_V03_FEMALE" device=""/>
 <part name="I20BSM1" library="bitSnap" deviceset="BITSNAP_V03_MALE" device=""/>
+<part name="U$1" library="LITTLEBITS" deviceset="OSHWCREDIT" device=""/>
+<part name="U$5" library="LITTLEBITS" deviceset="FRAME-LETTER-OHW" device="OHW"/>
 </parts>
 <sheets>
@@
 <instance part="I20U3" gate="G$1" x="193.04" y="93.98"/>
 <instance part="I20P1" gate="G$1" x="111.76" y="71.12" rot="MR270"/>
-<instance part="FRAME1" gate="G$1" x="0" y="0"/>
-<instance part="FRAME1" gate="G$2" x="147.32" y="0"/>
 <instance part="I20R1" gate="G$1" x="99.06" y="116.84"/>
 <instance part="I20R2" gate="G$1" x="86.36" y="96.52" rot="R180"/>
@@
 <attribute name="VALUE" x="166.624" y="124.841" size="1.778" layer="96"/>
 </instance>
-<instance part="U$28" gate="G$1" x="63.5" y="12.7"/>
 <instance part="U$29" gate="G$1" x="132.08" y="12.7"/>
 <instance part="I20Q1" gate="A" x="165.1" y="116.84"/>
@@
 <instance part="I20BSF1" gate="G$1" x="208.28" y="88.9"/>
 <instance part="I20BSM1" gate="G$1" x="33.02" y="91.44"/>
+<instance part="U$1" gate="G$1" x="68.58" y="7.62"/>
+<instance part="U$5" gate="G$1" x="0" y="0"/>
+<instance part="U$5" gate="G$2" x="147.32" y="0"/>
 </instances>
 <busses>
@@
 </schematic>
 </drawing>
+<compatibility>
+<note version="6.3" minversion="6.2.2" severity="warning">
+Since Version 6.2.2 text objects can contain more than one line,
+which will not be processed correctly with this version.
+</note>
+</compatibility>
 </eagle>

Commit message: Updated license text
Changed lines of the file:
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@@
 <part name="I20BSF1" library="bitSnap" deviceset="BITSNAP_V03_FEMALE" device=""/>
 <part name="I20BSM1" library="bitSnap" deviceset="BITSNAP_V03_MALE" device=""/>
+<part name="U$5" library="LITTLEBITS" deviceset="FRAME-LETTER-OHW" device="OHW"/>
 <part name="U$1" library="LITTLEBITS" deviceset="OSHWCREDIT" device=""/>
-<part name="U$5" library="LITTLEBITS" deviceset="FRAME-LETTER-OHW" device="OHW"/>
 </parts>
 <sheets>
@@
 <instance part="I20BSF1" gate="G$1" x="208.28" y="88.9"/>
 <instance part="I20BSM1" gate="G$1" x="33.02" y="91.44"/>
-<instance part="U$1" gate="G$1" x="68.58" y="7.62"/>
 <instance part="U$5" gate="G$1" x="0" y="0"/>
 <instance part="U$5" gate="G$2" x="147.32" y="0"/>
+<instance part="U$1" gate="G$1" x="48.26" y="10.16"/>
 </instances>
 <busses>
