File: INPUT/LB_BIT_i22_SEQUENCER/LB_BIT_i22_sequencer-v03(2_3)/LB_BIT_i22_sequencer-v03(rev2_3).sch (EAGLE design)
At the start: 61 parts

Commit message: Updated license text
Changed lines of the file:
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@@
 <?xml version="1.0" encoding="utf-8"?>
 <!DOCTYPE eagle SYSTEM "eagle.dtd">
-<eagle version="6.5.0">
+<eagle version="6.6.0">
 <drawing>
 <settings>
@@
 <instance part="I22TVS10" gate="G$1" x="81.28" y="86.36"/>
 <instance part="GND32" gate="1" x="45.72" y="73.66"/>
-<instance part="U$11" gate="G$1" x="134.62" y="10.16"/>
+<instance part="U$11" gate="G$1" x="99.06" y="10.16"/>
 <instance part="I22R5" gate="G$1" x="127" y="48.26" rot="R90"/>
 <instance part="GND34" gate="1" x="101.6" y="60.96" rot="R90"/>
 <instance part="U$14" gate="G$1" x="0" y="0"/>
 <instance part="U$14" gate="G$2" x="147.32" y="0"/>
-<instance part="U$15" gate="G$1" x="43.18" y="2.54"/>
+<instance part="U$15" gate="G$1" x="10.16" y="7.62"/>
 </instances>
 <busses>
