File: INPUT/LB_BIT_i8_MOTIONTRIGGER/LB_BIT_i18_MOTIONTRIGGER-v03(rev1)/LB_BIT_i18_MOTIONTRIGGER-v03(rev1).brd (EAGLE design)
At the start: 21.4 x 18.1 mm, 22 parts

Commit message: Updated licenses
Parts:
- removed FRAME1: FRAME-LETTER-OHWOHW, LITTLEBITS:FABDWG01-OHW
- removed U$9: LB_CREDITS_V2, LITTLEBITS:LB_CREDITS_V2
- added U$1: OSHWCREDIT, LITTLEBITS:OSHWCREDIT
- added U$2: FRAME-LETTER-OHWOHW, LITTLEBITS:FABDWG01-OHW
- moved U$8 48.5 mm to (-36.0, -59.7)
Changed lines of the file:
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@@
 <?xml version="1.0" encoding="utf-8"?>
 <!DOCTYPE eagle SYSTEM "eagle.dtd">
-<eagle version="6.1">
+<eagle version="6.6.0">
 <drawing>
 <settings>
@@
 <layer number="54" name="bGND_GNDA" color="7" fill="1" visible="yes" active="yes"/>
 <layer number="56" name="wert" color="7" fill="1" visible="yes" active="yes"/>
+<layer number="57" name="tCAD" color="7" fill="1" visible="no" active="no"/>
 <layer number="91" name="Nets" color="2" fill="1" visible="no" active="no"/>
 <layer number="92" name="Busses" color="1" fill="1" visible="no" active="no"/>
@@
 <layer number="145" name="DrillLegend_01-16" color="2" fill="9" visible="yes" active="yes"/>
 <layer number="146" name="DrillLegend_01-20" color="3" fill="9" visible="yes" active="yes"/>
+<layer number="150" name="Notes" color="7" fill="1" visible="yes" active="yes"/>
 <layer number="151" name="HeatSink" color="7" fill="1" visible="yes" active="yes"/>
 <layer number="152" name="_bDocu" color="7" fill="1" visible="yes" active="yes"/>
+<layer number="153" name="FabDoc1" color="6" fill="1" visible="no" active="no"/>
+<layer number="154" name="FabDoc2" color="2" fill="1" visible="no" active="no"/>
+<layer number="155" name="FabDoc3" color="7" fill="15" visible="no" active="no"/>
 <layer number="199" name="Contour" color="7" fill="1" visible="yes" active="yes"/>
 <layer number="200" name="200bmp" color="7" fill="1" visible="yes" active="yes"/>
@@
 <layer number="225" name="225bmp" color="26" fill="10" visible="yes" active="yes"/>
 <layer number="226" name="226bmp" color="27" fill="10" visible="yes" active="yes"/>
+<layer number="227" name="227bmp" color="7" fill="1" visible="yes" active="yes"/>
+<layer number="228" name="228bmp" color="7" fill="1" visible="yes" active="yes"/>
 <layer number="248" name="Housing" color="7" fill="1" visible="yes" active="yes"/>
 <layer number="249" name="Edge" color="7" fill="1" visible="yes" active="yes"/>
@@
 <wire x1="15.02" y1="23.092" x2="14.512" y2="23.6" width="0.1016" layer="146"/>
 <wire x1="14.512" y1="23.6" x2="15.02" y2="24.108" width="0.1016" layer="146"/>
-<dimension x1="3.8" y1="26.5" x2="16.6" y2="26.5" x3="10.2" y3="37.7" layer="47" dtype="horizontal"/>
-<dimension x1="20.4" y1="22" x2="0" y2="22" x3="10.2" y3="44.9" layer="47" dtype="horizontal"/>
-<dimension x1="-0.5" y1="4.5" x2="-0.5" y2="21.5" x3="-4.2" y3="13" layer="47" dtype="vertical"/>
-<dimension x1="3.3" y1="0" x2="3.3" y2="26" x3="-12.3" y3="13" layer="47" dtype="vertical"/>
-<dimension x1="4.35" y1="22.1" x2="16.05" y2="22.1" x3="10.2" y3="31.6" layer="47" dtype="horizontal"/>
+<dimension x1="3.8" y1="26.5" x2="16.6" y2="26.5" x3="10.2" y3="37.7" textsize="3.5" layer="47" dtype="horizontal"/>
+<dimension x1="20.4" y1="22" x2="0" y2="22" x3="10.2" y3="44.9" textsize="3.5" layer="47" dtype="horizontal"/>
+<dimension x1="-0.5" y1="4.5" x2="-0.5" y2="21.5" x3="-4.2" y3="13" textsize="3.5" layer="47" dtype="vertical"/>
+<dimension x1="3.3" y1="0" x2="3.3" y2="26" x3="-12.3" y3="13" textsize="3.5" layer="47" dtype="vertical"/>
+<dimension x1="4.35" y1="22.1" x2="16.05" y2="22.1" x3="10.2" y3="31.6" textsize="3.5" layer="47" dtype="horizontal"/>
 <text x="-5.9" y="52.25" size="1.778" layer="46">1mm DIA. ROUTER PATH</text>
 <text x="18.05" y="14.35" size="1.2" layer="21" font="vector" rot="SR270">i18</text>
@@
 </class>
 </classes>
-<designrules>
+<designrules name="default">
 <description language="en">&lt;b&gt;EAGLE Design Rules&lt;/b&gt;
 &lt;p&gt;
@@
 <attribute name="VALUE" x="17.552" y="5.3265" size="0.4064" layer="28" font="vector" rot="MR90"/>
 </element>
-<element name="U$8" library="SparkFun_NEW" package="OSHW-LOGO-L" value="OSHW-LOGOL" x="-18.95" y="-14.26"/>
-<element name="U$9" library="LITTLEBITS" package="LB_CREDITS_V2" value="LB_CREDITS_V2" x="-2.1" y="-16.7"/>
+<element name="U$8" library="SparkFun_NEW" package="OSHW-LOGO-L" value="OSHW-LOGOL" x="-36" y="-59.71"/>
 <element name="I18C4" library="SparkFun" package="0603-CAP" value="0.1uF" x="6.559" y="13.077" smashed="yes" rot="MR90">
 <attribute name="NAME" x="7.512" y="14.571" size="0.4064" layer="26" font="vector" rot="MR0"/>
@@
 <element name="I18BSM" library="bitSnap" package="BITSNAP_V03_MALE" value="BITSNAP_V03_MALE" x="16.65" y="26.1" rot="R180"/>
 <element name="I18BSF" library="bitSnap" package="BITSNAP_V03_FEMALE" value="BITSNAP_V03_FEMALE" x="3.75" y="0"/>
-<element name="FRAME1" library="LITTLEBITS" package="FABDWG01-OHW" value="FRAME-LETTER-OHWOHW" x="-61.84" y="7.13"/>
+<element name="U$1" library="LITTLEBITS" package="OSHWCREDIT" value="OSHWCREDIT" x="-94.3" y="-64.7"/>
+<element name="U$2" library="LITTLEBITS" package="FABDWG01-OHW" value="FRAME-LETTER-OHWOHW" x="0" y="0"/>
 </elements>
 <signals>
@@
 </board>
 </drawing>
+<compatibility>
+<note version="6.3" minversion="6.2.2" severity="warning">
+Since Version 6.2.2 text objects can contain more than one line,
+which will not be processed correctly with this version.
+</note>
+</compatibility>
 </eagle>

Commit message: Updated license text
Parts:
- I18U2: value LV321SOT-235 -> LV321SOT23-5
- moved U$8 10.4 mm to (-32.8, -69.6)
Changed lines of the file:
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@@
 </element>
 <element name="I18R3" library="SparkFun" package="0603-RES" value="100K" x="2.42" y="7.2125" rot="MR180"/>
-<element name="I18U2" library="LITTLEBITS" package="SOT23-5" value="LV321SOT-235" x="15.9075" y="7.65" smashed="yes" rot="MR270">
+<element name="I18U2" library="LITTLEBITS" package="SOT23-5" value="LV321SOT23-5" x="15.9075" y="7.65" smashed="yes" rot="MR270">
 <attribute name="NAME" x="16.4835" y="8.489" size="0.4064" layer="26" rot="MR270"/>
 <attribute name="VALUE" x="15.5615" y="9.112" size="0.3048" layer="28" rot="MR270"/>
@@
 <attribute name="VALUE" x="17.552" y="5.3265" size="0.4064" layer="28" font="vector" rot="MR90"/>
 </element>
-<element name="U$8" library="SparkFun_NEW" package="OSHW-LOGO-L" value="OSHW-LOGOL" x="-36" y="-59.71"/>
+<element name="U$8" library="SparkFun_NEW" package="OSHW-LOGO-L" value="OSHW-LOGOL" x="-32.8" y="-69.56"/>
 <element name="I18C4" library="SparkFun" package="0603-CAP" value="0.1uF" x="6.559" y="13.077" smashed="yes" rot="MR90">
 <attribute name="NAME" x="7.512" y="14.571" size="0.4064" layer="26" font="vector" rot="MR0"/>
