File: OUTPUT/LB_BIT_o16_LIGHTWIRE/LB_BIT_o16_LIGHTWIRE-v03(rev2)/LB_BIT_o16_LIGHTWIRE-v03(rev2).brd (EAGLE design)
At the start: 21.4 x 24.7 mm, 22 parts

Commit message: Updated licenses
Parts:
- U$2: value LB_CREDITS_V2 -> OSHWCREDIT; device LITTLEBITS:LB_CREDITS_V2 -> LITTLEBITS:OSHWCREDIT
- moved U$5 193.8 mm to (0.00, 0.00)
- moved U$2 88.3 mm to (-91.8, -65.3)
- moved U$1 42.7 mm to (-35.3, -59.9)
Changed lines of the file:
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@@
 <?xml version="1.0" encoding="utf-8"?>
 <!DOCTYPE eagle SYSTEM "eagle.dtd">
-<eagle version="6.1">
+<eagle version="6.6.0">
 <drawing>
 <settings>
@@
 <layer number="54" name="bGND_GNDA" color="7" fill="1" visible="yes" active="yes"/>
 <layer number="56" name="wert" color="7" fill="1" visible="yes" active="yes"/>
+<layer number="57" name="tCAD" color="7" fill="1" visible="no" active="no"/>
 <layer number="91" name="Nets" color="2" fill="1" visible="no" active="no"/>
 <layer number="92" name="Busses" color="1" fill="1" visible="no" active="no"/>
@@
 <layer number="145" name="DrillLegend_01-16" color="2" fill="9" visible="yes" active="yes"/>
 <layer number="146" name="DrillLegend_01-20" color="3" fill="9" visible="yes" active="yes"/>
+<layer number="150" name="Notes" color="7" fill="1" visible="yes" active="yes"/>
 <layer number="151" name="HeatSink" color="7" fill="1" visible="yes" active="yes"/>
 <layer number="152" name="_bDocu" color="7" fill="1" visible="yes" active="yes"/>
+<layer number="153" name="FabDoc1" color="6" fill="1" visible="no" active="no"/>
+<layer number="154" name="FabDoc2" color="2" fill="1" visible="no" active="no"/>
+<layer number="155" name="FabDoc3" color="7" fill="15" visible="no" active="no"/>
 <layer number="199" name="Contour" color="7" fill="1" visible="yes" active="yes"/>
 <layer number="200" name="200bmp" color="7" fill="1" visible="yes" active="yes"/>
@@
 <layer number="225" name="225bmp" color="26" fill="10" visible="yes" active="yes"/>
 <layer number="226" name="226bmp" color="27" fill="10" visible="yes" active="yes"/>
+<layer number="227" name="227bmp" color="7" fill="1" visible="yes" active="yes"/>
+<layer number="228" name="228bmp" color="7" fill="1" visible="yes" active="yes"/>
 <layer number="248" name="Housing" color="7" fill="1" visible="yes" active="yes"/>
 <layer number="249" name="Edge" color="7" fill="1" visible="yes" active="yes"/>
@@
 <hole x="-11.2" y="9.35" drill="1.5"/>
 <hole x="5.2" y="28.8" drill="1.5"/>
-<dimension x1="-13.2" y1="7.35" x2="-13.2" y2="11.35" x3="-15.05" y3="9.35" layer="51"/>
-<dimension x1="-11.2" y1="7.35" x2="-11.2" y2="9.35" x3="-20.9" y3="8.35" layer="51"/>
+<dimension x1="-13.2" y1="7.35" x2="-13.2" y2="11.35" x3="-15.05" y3="9.35" textsize="3.5" layer="51"/>
+<dimension x1="-11.2" y1="7.35" x2="-11.2" y2="9.35" x3="-20.9" y3="8.35" textsize="3.5" layer="51"/>
 <text x="6.75" y="10.8" size="0.8128" layer="16" font="vector" ratio="12" rot="MR270">rev2</text>
 <wire x1="-13.2" y1="31.55" x2="-13.7" y2="31.55" width="1" layer="46"/>
@@
 <wire x1="7.7" y1="6.85" x2="7.7" y2="31.55" width="1" layer="46"/>
 <wire x1="7.7" y1="31.55" x2="7.2" y2="31.55" width="1" layer="46"/>
-<dimension x1="-9.4" y1="36.05" x2="3.4" y2="36.05" x3="-3" y3="47.25" layer="47" dtype="horizontal"/>
-<dimension x1="7.2" y1="31.55" x2="-13.2" y2="31.55" x3="-3" y3="54.7" layer="47" dtype="horizontal"/>
-<dimension x1="-13.7" y1="7.35" x2="-13.7" y2="31.05" x3="-17.4" y3="19.2" layer="47" dtype="vertical"/>
-<dimension x1="-9.9" y1="2.85" x2="-9.9" y2="35.55" x3="-25.5" y3="19.2" layer="47" dtype="vertical"/>
-<dimension x1="-8.85" y1="31.55" x2="2.85" y2="31.55" x3="-3" y3="40.95" layer="47" dtype="horizontal"/>
+<dimension x1="-9.4" y1="36.05" x2="3.4" y2="36.05" x3="-3" y3="47.25" textsize="3.5" layer="47" dtype="horizontal"/>
+<dimension x1="7.2" y1="31.55" x2="-13.2" y2="31.55" x3="-3" y3="54.7" textsize="3.5" layer="47" dtype="horizontal"/>
+<dimension x1="-13.7" y1="7.35" x2="-13.7" y2="31.05" x3="-17.4" y3="19.2" textsize="3.5" layer="47" dtype="vertical"/>
+<dimension x1="-9.9" y1="2.85" x2="-9.9" y2="35.55" x3="-25.5" y3="19.2" textsize="3.5" layer="47" dtype="vertical"/>
+<dimension x1="-8.85" y1="31.55" x2="2.85" y2="31.55" x3="-3" y3="40.95" textsize="3.5" layer="47" dtype="horizontal"/>
 <wire x1="-3.35" y1="23.508" x2="-3.35" y2="22.492" width="0.1016" layer="145"/>
 <wire x1="-3.858" y1="23" x2="-2.842" y2="23" width="0.1016" layer="145"/>
@@
 <wire x1="4.692" y1="28.8" x2="5.2" y2="29.308" width="0.1016" layer="146"/>
 <text x="-19.7" y="-5.75" size="1.778" layer="46">1mm DIA. ROUTER PATH</text>
-<text x="-40.6" y="-42.6" size="1.778" layer="50">o16 LIGHT WIRE BIT PCB</text>
-<text x="27.4" y="-38.6" size="1.778" layer="50">2</text>
+<text x="-9.55" y="-47.65" size="1.778" layer="50">o16 LIGHT WIRE BIT PCB</text>
+<text x="56.1" y="-43.9" size="1.778" layer="50">2</text>
 <text x="5.15" y="26.45" size="1.3" layer="21" font="vector" rot="SR270">o16 light wire</text>
 </plain>
@@
 </class>
 </classes>
-<designrules>
+<designrules name="default">
 <description language="en">&lt;b&gt;EAGLE Design Rules&lt;/b&gt;
 &lt;p&gt;
@@
 <attribute name="NAME" x="-1.714" y="25.411" size="0.4064" layer="25"/>
 <attribute name="VALUE" x="-2.348" y="23.859" size="0.4064" layer="27" rot="R90"/>
+<attribute name="LB_PN" value="" x="-0.825" y="24.645" size="1.778" layer="27" display="off"/>
 </element>
 <element name="O16R4" library="SparkFun" package="0603-RES" value="10K" x="3.35" y="13" smashed="yes" rot="R270">
@@
 <attribute name="VALUE" x="-7.5075" y="23.6695" size="0.4064" layer="27"/>
 </element>
-<element name="U$1" library="SparkFun_NEW" package="OSHW-LOGO-L" value="OSHW-LOGOL" x="-36.12" y="-17.26"/>
-<element name="U$2" library="LITTLEBITS" package="LB_CREDITS_V2" value="LB_CREDITS_V2" x="-15.22" y="-21.25"/>
+<element name="U$1" library="SparkFun_NEW" package="OSHW-LOGO-L" value="OSHW-LOGOL" x="-35.27" y="-59.91"/>
 <element name="O16BSM1" library="bitSnap" package="BITSNAP_V03_MALE" value="BITSNAP_V03_MALE" x="3.45" y="35.55" rot="R180"/>
 <element name="O16BSF1" library="bitSnap" package="BITSNAP_V03_FEMALE" value="BITSNAP_V03_FEMALE" x="-9.45" y="2.85"/>
@@
 </element>
 <element name="O16JP1" library="SparkFun" package="S2B-PH" value="" x="-6.45" y="19.2" rot="R90"/>
-<element name="U$5" library="LITTLEBITS" package="FABDWG01-OHW" value="FRAME-LETTER-OHWOHW" x="-180.55" y="-70.45"/>
+<element name="U$5" library="LITTLEBITS" package="FABDWG01-OHW" value="FRAME-LETTER-OHWOHW" x="0" y="0"/>
+<element name="U$2" library="LITTLEBITS" package="OSHWCREDIT" value="OSHWCREDIT" x="-91.8" y="-65.3"/>
 </elements>
 <signals>
@@
 </board>
 </drawing>
+<compatibility>
+<note version="6.3" minversion="6.2.2" severity="warning">
+Since Version 6.2.2 text objects can contain more than one line,
+which will not be processed correctly with this version.
+</note>
+</compatibility>
 </eagle>

Commit message: Updated license text
Parts:
- moved U$1 9.95 mm to (-31.0, -68.9)
Changed lines of the file:
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@@
 <attribute name="VALUE" x="-7.5075" y="23.6695" size="0.4064" layer="27"/>
 </element>
-<element name="U$1" library="SparkFun_NEW" package="OSHW-LOGO-L" value="OSHW-LOGOL" x="-35.27" y="-59.91"/>
+<element name="U$1" library="SparkFun_NEW" package="OSHW-LOGO-L" value="OSHW-LOGOL" x="-31.02" y="-68.91"/>
 <element name="O16BSM1" library="bitSnap" package="BITSNAP_V03_MALE" value="BITSNAP_V03_MALE" x="3.45" y="35.55" rot="R180"/>
 <element name="O16BSF1" library="bitSnap" package="BITSNAP_V03_FEMALE" value="BITSNAP_V03_FEMALE" x="-9.45" y="2.85"/>
