File: OUTPUT/LB_BIT_o21_NUMBER/LB_BIT_o21_number-v03(rev3_3)/LB_BIT_o21_number-v03(rev3_3).brd (EAGLE design)
At the start: 21.4 x 37.9 mm, 22 parts

Commit message: Updated license text
Parts:
- moved U$7 3.58 mm to (-92.7, -63.3)
Changed lines of the file:
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@@
 <?xml version="1.0" encoding="utf-8"?>
 <!DOCTYPE eagle SYSTEM "eagle.dtd">
-<eagle version="7.0.0">
+<eagle version="6.6.0">
 <drawing>
 <settings>
@@
 <pass name="Default">
 <param name="RoutingGrid" value="50mil"/>
-<param name="AutoGrid" value="1"/>
-<param name="Efforts" value="0"/>
-<param name="TopRouterVariant" value="1"/>
 <param name="tpViaShape" value="round"/>
 <param name="PrefDir.1" value="|"/>
@@
 <attribute name="LB_PN" value="?" x="8.65" y="32.3" size="1.778" layer="28" rot="MR180" display="off"/>
 <attribute name="V_OPERATION" value="5V" x="8.65" y="32.3" size="1.778" layer="28" rot="MR180" display="off"/>
-<attribute name="IEC_ESD_PROT" value="+/-18kV" x="8.65" y="32.3" size="1.778" layer="28" rot="MR180" display="off"/>
 <attribute name="V_CLAMP" value="?" x="8.65" y="32.3" size="1.778" layer="28" rot="MR180" display="off"/>
 <attribute name="NAME" x="7.461" y="34.384" size="0.4064" layer="26" rot="MR270"/>
 <attribute name="VALUE" x="6.034" y="31.647" size="0.4064" layer="28" rot="MR180"/>
+<attribute name="MPN" value="ESD9B5.0ST5G" x="8.65" y="32.3" size="1.778" layer="28" rot="MR180" display="off"/>
+<attribute name="IEC_ESD_PROT0" value="+/-18kV" x="8.65" y="32.3" size="1.778" layer="28" rot="MR180" display="off"/>
 </element>
 <element name="O21R2" library="LITTLEBITS" package="RES-0603" value="1M" x="4.35" y="32.35" smashed="yes" rot="MR0">
@@
 <attribute name="VALUE" x="13.284" y="35.743" size="0.4064" layer="28" font="vector" rot="MR270"/>
 </element>
-<element name="U$7" library="LITTLEBITS" package="OSHWCREDIT" value="OSHWCREDIT" x="-90.6" y="-66.2"/>
+<element name="U$7" library="LITTLEBITS" package="OSHWCREDIT" value="OSHWCREDIT" x="-92.7" y="-63.3"/>
 <element name="U$16" library="LITTLEBITS" package="FABDWG01-OHW" value="FRAME-LETTER-OHWOHW" x="0" y="0"/>
 </elements>
