File: OUTPUT/LB_BIT_o3_RGBLED/LB_o3_RGB_LED-v03(rev2)/LB_o3_RGB_LED-v03(rev2).sch (EAGLE design)
At the start: 14 parts

Commit message: Updated licenses
Parts:
- removed FRAME1: FRAME-LETTER-OHWOHW, LITTLEBITS:FRAME-LETTER-OHWOHW
- added U$2: OSHWCREDIT, LITTLEBITS:OSHWCREDIT
- U$1: value OSHWCREDIT -> FRAME-LETTER-OHWOHW; device LITTLEBITS:OSHWCREDIT -> LITTLEBITS:FRAME-LETTER-OHWOHW
Changed lines of the file:
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@@
 <?xml version="1.0" encoding="utf-8"?>
 <!DOCTYPE eagle SYSTEM "eagle.dtd">
-<eagle version="6.5.0">
+<eagle version="6.6.0">
 <drawing>
 <settings>
@@
 <layer number="54" name="bGND_GNDA" color="1" fill="9" visible="no" active="no"/>
 <layer number="56" name="wert" color="7" fill="1" visible="no" active="no"/>
+<layer number="57" name="tCAD" color="7" fill="1" visible="no" active="no"/>
 <layer number="91" name="Nets" color="2" fill="1" visible="yes" active="yes"/>
 <layer number="92" name="Busses" color="1" fill="1" visible="yes" active="yes"/>
@@
 <layer number="145" name="DrillLegend_01-16" color="2" fill="9" visible="yes" active="yes"/>
 <layer number="146" name="DrillLegend_01-20" color="3" fill="9" visible="yes" active="yes"/>
+<layer number="150" name="Notes" color="7" fill="1" visible="yes" active="yes"/>
 <layer number="151" name="HeatSink" color="7" fill="1" visible="yes" active="yes"/>
 <layer number="152" name="_bDocu" color="7" fill="1" visible="yes" active="yes"/>
+<layer number="153" name="FabDoc1" color="6" fill="1" visible="no" active="no"/>
+<layer number="154" name="FabDoc2" color="2" fill="1" visible="no" active="no"/>
+<layer number="155" name="FabDoc3" color="7" fill="15" visible="no" active="no"/>
 <layer number="199" name="Contour" color="7" fill="1" visible="yes" active="yes"/>
 <layer number="200" name="200bmp" color="1" fill="10" visible="no" active="no"/>
@@
 <layer number="225" name="225bmp" color="26" fill="10" visible="no" active="yes"/>
 <layer number="226" name="226bmp" color="27" fill="10" visible="no" active="yes"/>
+<layer number="227" name="227bmp" color="7" fill="1" visible="yes" active="yes"/>
+<layer number="228" name="228bmp" color="7" fill="1" visible="yes" active="yes"/>
 <layer number="248" name="Housing" color="7" fill="1" visible="yes" active="yes"/>
 <layer number="249" name="Edge" color="7" fill="1" visible="yes" active="yes"/>
@@
 </classes>
 <parts>
-<part name="FRAME1" library="LITTLEBITS" deviceset="FRAME-LETTER-OHW" device="OHW"/>
 <part name="GND2" library="supply1" deviceset="GND" device=""/>
 <part name="O3R4" library="SparkFun" deviceset="RESISTOR" device="0603-RES" value="220"/>
@@
 <part name="O3D1" library="LITTLEBITS" deviceset="LED-RGB-SUN_XZMDKCBDDG45S" device=""/>
 <part name="O3U1" library="LITTLEBITS" deviceset="LV321" device="SOT-235"/>
-<part name="U$1" library="LITTLEBITS" deviceset="OSHWCREDIT" device=""/>
 <part name="O3BSM1" library="bitSnap" deviceset="BITSNAP_V03_MALE" device=""/>
 <part name="O3BSF1" library="bitSnap" deviceset="BITSNAP_V03_FEMALE" device=""/>
+<part name="U$1" library="LITTLEBITS" deviceset="FRAME-LETTER-OHW" device="OHW"/>
+<part name="U$2" library="LITTLEBITS" deviceset="OSHWCREDIT" device=""/>
 </parts>
 <sheets>
@@
 </plain>
 <instances>
-<instance part="FRAME1" gate="G$1" x="0" y="0"/>
-<instance part="FRAME1" gate="G$2" x="147.32" y="0"/>
 <instance part="GND2" gate="1" x="81.28" y="68.58"/>
 <instance part="O3R4" gate="G$1" x="106.68" y="93.98"/>
@@
 <instance part="O3D1" gate="G$1" x="124.46" y="76.2"/>
 <instance part="O3U1" gate="G$1" x="134.62" y="134.62"/>
-<instance part="U$1" gate="G$1" x="35.56" y="10.16"/>
 <instance part="O3BSM1" gate="G$1" x="96.52" y="114.3"/>
 <instance part="O3BSF1" gate="G$1" x="154.94" y="114.3"/>
+<instance part="U$1" gate="G$1" x="0" y="0"/>
+<instance part="U$1" gate="G$2" x="147.32" y="0"/>
+<instance part="U$2" gate="G$1" x="40.64" y="10.16"/>
 </instances>
 <busses>
@@
 </schematic>
 </drawing>
+<compatibility>
+<note version="6.3" minversion="6.2.2" severity="warning">
+Since Version 6.2.2 text objects can contain more than one line,
+which will not be processed correctly with this version.
+</note>
+</compatibility>
 </eagle>

Commit message: Updated license text
Parts:
- O3U1: value LV321SOT-235 -> LV321SOT23-5; device LITTLEBITS:LV321SOT-235 -> LITTLEBITS:LV321SOT23-5
Changed lines of the file:
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@@
 <part name="GND3" library="SparkFun" deviceset="GND" device=""/>
 <part name="O3D1" library="LITTLEBITS" deviceset="LED-RGB-SUN_XZMDKCBDDG45S" device=""/>
-<part name="O3U1" library="LITTLEBITS" deviceset="LV321" device="SOT-235"/>
+<part name="O3U1" library="LITTLEBITS" deviceset="LV321" device="SOT23-5"/>
 <part name="O3BSM1" library="bitSnap" deviceset="BITSNAP_V03_MALE" device=""/>
 <part name="O3BSF1" library="bitSnap" deviceset="BITSNAP_V03_FEMALE" device=""/>
