File: OUTPUT/LB_BIT_o4_VIBRATIONMOTOR/LB_o4_Vibration_Motor-v03(rev2)/LB_o4_Vibration_Motor-v03(rev2).sch (EAGLE design)
At the start: 12 parts

Commit message: Updated licenses
Parts:
- removed U$6: OSHWCREDIT, LITTLEBITS:OSHWCREDIT
- added U$1: OSHWCREDIT, LITTLEBITS:OSHWCREDIT
- renumbered FRAME1 to U$2
Changed lines of the file:
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@@
 <?xml version="1.0" encoding="utf-8"?>
 <!DOCTYPE eagle SYSTEM "eagle.dtd">
-<eagle version="6.1">
+<eagle version="6.6.0">
 <drawing>
 <settings>
@@
 <layer number="54" name="bGND_GNDA" color="1" fill="9" visible="no" active="no"/>
 <layer number="56" name="wert" color="7" fill="1" visible="no" active="no"/>
+<layer number="57" name="tCAD" color="7" fill="1" visible="no" active="no"/>
 <layer number="91" name="Nets" color="2" fill="1" visible="yes" active="yes"/>
 <layer number="92" name="Busses" color="1" fill="1" visible="yes" active="yes"/>
@@
 <layer number="145" name="DrillLegend_01-16" color="2" fill="9" visible="yes" active="yes"/>
 <layer number="146" name="DrillLegend_01-20" color="3" fill="9" visible="yes" active="yes"/>
+<layer number="150" name="Notes" color="7" fill="1" visible="yes" active="yes"/>
 <layer number="151" name="HeatSink" color="7" fill="1" visible="yes" active="yes"/>
 <layer number="152" name="_bDocu" color="7" fill="1" visible="yes" active="yes"/>
+<layer number="153" name="FabDoc1" color="6" fill="1" visible="no" active="no"/>
+<layer number="154" name="FabDoc2" color="2" fill="1" visible="no" active="no"/>
+<layer number="155" name="FabDoc3" color="7" fill="15" visible="no" active="no"/>
 <layer number="199" name="Contour" color="7" fill="1" visible="yes" active="yes"/>
 <layer number="200" name="200bmp" color="1" fill="10" visible="no" active="no"/>
@@
 <layer number="225" name="225bmp" color="26" fill="10" visible="no" active="yes"/>
 <layer number="226" name="226bmp" color="27" fill="10" visible="no" active="yes"/>
+<layer number="227" name="227bmp" color="7" fill="1" visible="yes" active="yes"/>
+<layer number="228" name="228bmp" color="7" fill="1" visible="yes" active="yes"/>
 <layer number="248" name="Housing" color="7" fill="1" visible="yes" active="yes"/>
 <layer number="249" name="Edge" color="7" fill="1" visible="yes" active="yes"/>
@@
 <part name="O4R1" library="SparkFun" deviceset="RESISTOR" device="0603-RES" value="330k"/>
 <part name="O4D1" library="SparkFun" deviceset="DIODE" device="SOT23" value="BAS16"/>
-<part name="FRAME1" library="LITTLEBITS" deviceset="FRAME-LETTER-OHW" device="OHW"/>
 <part name="O4JP1" library="LITTLEBITS" deviceset="JST-MICRO-2P" device="" value="MOTOR"/>
 <part name="O4C1" library="SparkFun" deviceset="CAP" device="0603-CAP" value="0.1uF"/>
@@
 <part name="P+1" library="SparkFun" deviceset="VCC" device=""/>
 <part name="O4U1" library="LITTLEBITS" deviceset="LV321" device="SOT-235"/>
-<part name="U$6" library="LITTLEBITS" deviceset="OSHWCREDIT" device=""/>
 <part name="O4BSM1" library="bitSnap" deviceset="BITSNAP_V03_MALE" device=""/>
 <part name="O4BSF1" library="bitSnap" deviceset="BITSNAP_V03_FEMALE" device=""/>
 <part name="GND2" library="LITTLEBITS" deviceset="GND" device=""/>
 <part name="P+2" library="SparkFun" deviceset="VCC" device=""/>
+<part name="U$1" library="LITTLEBITS" deviceset="OSHWCREDIT" device=""/>
+<part name="U$2" library="LITTLEBITS" deviceset="FRAME-LETTER-OHW" device="OHW"/>
 </parts>
 <sheets>
@@
 <attribute name="VALUE" x="163.8554" y="90.678" size="1.778" layer="96" rot="R90"/>
 </instance>
-<instance part="FRAME1" gate="G$1" x="0" y="0"/>
-<instance part="FRAME1" gate="G$2" x="147.32" y="0"/>
 <instance part="O4JP1" gate="G$1" x="134.62" y="86.36" smashed="yes">
 <attribute name="NAME" x="134.366" y="95.25" size="1.778" layer="95"/>
@@
 <attribute name="VALUE" x="107.95" y="86.36" size="1.778" layer="96"/>
 </instance>
-<instance part="U$6" gate="G$1" x="35.56" y="7.62"/>
 <instance part="O4BSM1" gate="G$1" x="63.5" y="96.52"/>
 <instance part="O4BSF1" gate="G$1" x="170.18" y="96.52"/>
 <instance part="GND2" gate="1" x="121.92" y="78.74"/>
 <instance part="P+2" gate="1" x="121.92" y="114.3"/>
+<instance part="U$1" gate="G$1" x="68.58" y="5.08"/>
+<instance part="U$2" gate="G$1" x="0" y="0"/>
+<instance part="U$2" gate="G$2" x="147.32" y="0"/>
 </instances>
 <busses>
@@
 </schematic>
 </drawing>
+<compatibility>
+<note version="6.3" minversion="6.2.2" severity="warning">
+Since Version 6.2.2 text objects can contain more than one line,
+which will not be processed correctly with this version.
+</note>
+</compatibility>
 </eagle>

Commit message: Updated license text
Parts:
- O4U1: value LV321SOT-235 -> LV321SOT23-5; device LITTLEBITS:LV321SOT-235 -> LITTLEBITS:LV321SOT23-5
Changed lines of the file:
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@@
 <part name="GND1" library="SparkFun" deviceset="GND" device=""/>
 <part name="P+1" library="SparkFun" deviceset="VCC" device=""/>
-<part name="O4U1" library="LITTLEBITS" deviceset="LV321" device="SOT-235"/>
+<part name="O4U1" library="LITTLEBITS" deviceset="LV321" device="SOT23-5"/>
 <part name="O4BSM1" library="bitSnap" deviceset="BITSNAP_V03_MALE" device=""/>
 <part name="O4BSF1" library="bitSnap" deviceset="BITSNAP_V03_FEMALE" device=""/>
@@
 <instance part="GND2" gate="1" x="121.92" y="78.74"/>
 <instance part="P+2" gate="1" x="121.92" y="114.3"/>
-<instance part="U$1" gate="G$1" x="68.58" y="5.08"/>
+<instance part="U$1" gate="G$1" x="48.26" y="7.62"/>
 <instance part="U$2" gate="G$1" x="0" y="0"/>
 <instance part="U$2" gate="G$2" x="147.32" y="0"/>
