File: OUTPUT/LB_BIT_o5_DCMOTOR/LB_BIT_o5_DCMOTOR-v02(rev1)/LB_BIT_o5_DCMOTOR-v02(rev1).brd (EAGLE design)
At the start: 20.3 x 58.4 mm, 47 parts

Commit message: Updated licenses
Parts:
- U$6: value LB_CREDITS_V2 -> OSHWCREDIT; device LITTLEBITS:LB_CREDITS_V2 -> LITTLEBITS:OSHWCREDIT
- moved U$6 19.4 mm to (-16.5, -24.1)
Changed lines of the file:
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@@
 <?xml version="1.0" encoding="utf-8"?>
 <!DOCTYPE eagle SYSTEM "eagle.dtd">
-<eagle version="6.2">
+<eagle version="6.6.0">
 <drawing>
 <settings>
@@
 <layer number="54" name="bGND_GNDA" color="1" fill="9" visible="no" active="no"/>
 <layer number="56" name="wert" color="7" fill="1" visible="yes" active="yes"/>
+<layer number="57" name="tCAD" color="7" fill="1" visible="no" active="no"/>
 <layer number="91" name="Nets" color="2" fill="1" visible="no" active="no"/>
 <layer number="92" name="Busses" color="1" fill="1" visible="no" active="no"/>
@@
 <layer number="106" name="bPlate" color="7" fill="1" visible="yes" active="yes"/>
 <layer number="107" name="Crop" color="7" fill="1" visible="yes" active="yes"/>
+<layer number="108" name="fp8" color="7" fill="1" visible="yes" active="yes"/>
+<layer number="109" name="fp9" color="7" fill="1" visible="yes" active="yes"/>
+<layer number="110" name="fp0" color="7" fill="1" visible="yes" active="yes"/>
+<layer number="111" name="LB_TEXT" color="13" fill="1" visible="yes" active="yes"/>
+<layer number="112" name="tSilk" color="7" fill="1" visible="yes" active="yes"/>
 <layer number="116" name="Patch_BOT" color="9" fill="4" visible="yes" active="yes"/>
 <layer number="121" name="_tsilk" color="7" fill="1" visible="yes" active="yes"/>
 <layer number="122" name="_bsilk" color="7" fill="1" visible="yes" active="yes"/>
+<layer number="123" name="tTestmark" color="7" fill="1" visible="yes" active="yes"/>
+<layer number="124" name="bTestmark" color="7" fill="1" visible="yes" active="yes"/>
 <layer number="125" name="_tNames" color="7" fill="1" visible="yes" active="yes"/>
+<layer number="126" name="_bNames" color="7" fill="1" visible="yes" active="yes"/>
+<layer number="127" name="_tValues" color="7" fill="1" visible="yes" active="yes"/>
+<layer number="128" name="_bValues" color="7" fill="1" visible="yes" active="yes"/>
+<layer number="131" name="tAdjust" color="7" fill="1" visible="yes" active="yes"/>
+<layer number="132" name="bAdjust" color="7" fill="1" visible="yes" active="yes"/>
 <layer number="144" name="Drill_legend" color="7" fill="1" visible="yes" active="yes"/>
+<layer number="145" name="DrillLegend_01-16" color="2" fill="9" visible="yes" active="yes"/>
+<layer number="146" name="DrillLegend_01-20" color="3" fill="9" visible="yes" active="yes"/>
+<layer number="150" name="Notes" color="7" fill="1" visible="yes" active="yes"/>
 <layer number="151" name="HeatSink" color="7" fill="1" visible="yes" active="yes"/>
+<layer number="152" name="_bDocu" color="7" fill="1" visible="yes" active="yes"/>
+<layer number="153" name="FabDoc1" color="6" fill="1" visible="no" active="no"/>
+<layer number="154" name="FabDoc2" color="2" fill="1" visible="no" active="no"/>
+<layer number="155" name="FabDoc3" color="7" fill="15" visible="no" active="no"/>
+<layer number="199" name="Contour" color="7" fill="1" visible="yes" active="yes"/>
 <layer number="200" name="200bmp" color="1" fill="10" visible="no" active="no"/>
 <layer number="201" name="201bmp" color="2" fill="1" visible="no" active="no"/>
@@
 <layer number="223" name="223bmp" color="7" fill="1" visible="yes" active="yes"/>
 <layer number="224" name="224bmp" color="7" fill="1" visible="yes" active="yes"/>
+<layer number="225" name="225bmp" color="7" fill="1" visible="yes" active="yes"/>
+<layer number="226" name="226bmp" color="7" fill="1" visible="yes" active="yes"/>
+<layer number="227" name="227bmp" color="7" fill="1" visible="yes" active="yes"/>
+<layer number="228" name="228bmp" color="7" fill="1" visible="yes" active="yes"/>
+<layer number="248" name="Housing" color="7" fill="1" visible="yes" active="yes"/>
+<layer number="249" name="Edge" color="7" fill="1" visible="yes" active="yes"/>
 <layer number="250" name="Descript" color="3" fill="1" visible="no" active="no"/>
 <layer number="251" name="SMDround" color="12" fill="11" visible="no" active="no"/>
@@
 </class>
 </classes>
-<designrules>
+<designrules name="default">
 <description language="en">&lt;b&gt;EAGLE Design Rules&lt;/b&gt;
 &lt;p&gt;
@@
 <element name="U$60" library="littleBits_font" package="T" value="" x="0.762" y="13.589" rot="R270"/>
 <element name="U$4" library="SparkFun_NEW" package="OSHW-LOGO-L" value="OSHW-LOGOL" x="-12.7" y="-11.43"/>
-<element name="U$6" library="LITTLEBITS" package="LB_CREDITS_V2" value="LB_CREDITS_V2" x="0" y="-13.97"/>
+<element name="U$6" library="LITTLEBITS" package="OSHWCREDIT" value="OSHWCREDIT" x="-16.51" y="-24.13"/>
 </elements>
 <signals>
@@
 </board>
 </drawing>
+<compatibility>
+<note version="6.3" minversion="6.2.2" severity="warning">
+Since Version 6.2.2 text objects can contain more than one line,
+which will not be processed correctly with this version.
+</note>
+</compatibility>
 </eagle>

Commit message: Updated license text
Parts:
- U$1: device LITTLEBITS:SC70 -> LITTLEBITS:SC70-5
Changed lines of the file:
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@@
 <element name="O5BSM" library="bitSnap" package="BITSNAP_MALE" value="BITSNAP_MALE" x="19.05" y="58.42" rot="R180"/>
 <element name="O5BSF" library="bitSnap" package="BITSNAP_FEMALE" value="BITSNAP_FEMALE" x="1.27" y="0"/>
-<element name="O5D1" library="LITTLEBITS" package="SMA-DIODE" value="MRA140" x="15.875" y="45.4025" rot="R90"/>
-<element name="O5D2" library="LITTLEBITS" package="SMA-DIODE" value="MBRA140" x="13.0175" y="15.24" rot="R270"/>
+<element name="O5D1" library="LITTLEBITS" package="SMA-DIODE" value="MRA140" x="15.875" y="45.4025" rot="R90">
+<attribute name="LB_PN" value="" x="15.875" y="45.4025" size="1.778" layer="27" rot="R90" display="off"/>
+</element>
+<element name="O5D2" library="LITTLEBITS" package="SMA-DIODE" value="MBRA140" x="13.0175" y="15.24" rot="R270">
+<attribute name="LB_PN" value="" x="13.0175" y="15.24" size="1.778" layer="27" rot="R270" display="off"/>
+</element>
 <element name="O5C1" library="SparkFun" package="0603-CAP" value="0.1uF" x="1.905" y="8.89" rot="R270"/>
 <element name="U$8" library="ohw-logo" package="OSHW_FILLX150_NOTEXT" value="" x="8.509" y="52.959"/>
@@
 <element name="O5C3" library="SparkFun" package="0603-CAP" value="1nF" x="19.05" y="45.085" rot="R270"/>
 <element name="O5C4" library="SparkFun" package="0603-CAP" value="1nF" x="17.78" y="17.4625"/>
-<element name="U$1" library="LITTLEBITS" package="SC70" value="LV321" x="18.415" y="51.1175"/>
+<element name="U$1" library="LITTLEBITS" package="SC70-5" value="LV321" x="18.415" y="51.1175"/>
 <element name="U$2" library="littleBits_font" package="O" value="" x="18.796" y="10.541" rot="R270"/>
 <element name="U$3" library="littleBits_font" package="5" value="" x="18.4785" y="9.5885" rot="R270"/>
