File: OUTPUT/LB_BIT_o6_BUZZER/LB_BIT_o6_BUZZER-v03(3_3)/LB_BIT_o6_BUZZER-v03(3_3).brd (EAGLE design)
At the start: 21.4 x 24.7 mm, 14 parts

Commit message: Updated licenses
Parts:
- removed U$15: LB_CREDITS_V2, LITTLEBITS:LB_CREDITS_V2
- added U$2: OSHWCREDIT, LITTLEBITS:OSHWCREDIT
- moved U$1 166.8 mm to (0.00, 0.00)
- moved U$16 44.3 mm to (-33.4, -60.9)
Changed lines of the file:
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@@
 <?xml version="1.0" encoding="utf-8"?>
 <!DOCTYPE eagle SYSTEM "eagle.dtd">
-<eagle version="6.1">
+<eagle version="6.6.0">
 <drawing>
 <settings>
@@
 <layer number="54" name="bGND_GNDA" color="1" fill="9" visible="no" active="no"/>
 <layer number="56" name="wert" color="7" fill="1" visible="yes" active="yes"/>
+<layer number="57" name="tCAD" color="7" fill="1" visible="no" active="no"/>
 <layer number="91" name="Nets" color="2" fill="1" visible="no" active="no"/>
 <layer number="92" name="Busses" color="1" fill="1" visible="no" active="no"/>
@@
 <layer number="145" name="DrillLegend_01-16" color="2" fill="9" visible="yes" active="yes"/>
 <layer number="146" name="DrillLegend_01-20" color="3" fill="9" visible="yes" active="yes"/>
+<layer number="150" name="Notes" color="7" fill="1" visible="yes" active="yes"/>
 <layer number="151" name="HeatSink" color="7" fill="1" visible="yes" active="yes"/>
 <layer number="152" name="_bDocu" color="7" fill="1" visible="yes" active="yes"/>
+<layer number="153" name="FabDoc1" color="6" fill="1" visible="no" active="no"/>
+<layer number="154" name="FabDoc2" color="2" fill="1" visible="no" active="no"/>
+<layer number="155" name="FabDoc3" color="7" fill="15" visible="no" active="no"/>
 <layer number="199" name="Contour" color="7" fill="1" visible="yes" active="yes"/>
 <layer number="200" name="200bmp" color="1" fill="10" visible="no" active="no"/>
@@
 <layer number="225" name="225bmp" color="26" fill="10" visible="yes" active="yes"/>
 <layer number="226" name="226bmp" color="27" fill="10" visible="yes" active="yes"/>
+<layer number="227" name="227bmp" color="7" fill="1" visible="yes" active="yes"/>
+<layer number="228" name="228bmp" color="7" fill="1" visible="yes" active="yes"/>
 <layer number="248" name="Housing" color="7" fill="1" visible="yes" active="yes"/>
 <layer number="249" name="Edge" color="7" fill="1" visible="yes" active="yes"/>
@@
 <wire x1="20.9" y1="28.7" x2="20.9" y2="4" width="1" layer="46"/>
 <wire x1="-0.5" y1="4" x2="-0.5" y2="28.7" width="1" layer="46"/>
-<dimension x1="3.8" y1="33.2" x2="16.6" y2="33.2" x3="10.2" y3="44.4" layer="47" dtype="horizontal"/>
-<dimension x1="20.4" y1="28.7" x2="0" y2="28.7" x3="10.2" y3="51.85" layer="47" dtype="horizontal"/>
-<dimension x1="-0.5" y1="4.5" x2="-0.5" y2="28.2" x3="-4.2" y3="16.35" layer="47" dtype="vertical"/>
-<dimension x1="3.3" y1="0" x2="3.3" y2="32.7" x3="-12.3" y3="16.35" layer="47" dtype="vertical"/>
-<dimension x1="4.35" y1="28.7" x2="16.05" y2="28.7" x3="10.2" y3="38.1" layer="47" dtype="horizontal"/>
+<dimension x1="3.8" y1="33.2" x2="16.6" y2="33.2" x3="10.2" y3="44.4" textsize="3.5" layer="47" dtype="horizontal"/>
+<dimension x1="20.4" y1="28.7" x2="0" y2="28.7" x3="10.2" y3="51.85" textsize="3.5" layer="47" dtype="horizontal"/>
+<dimension x1="-0.5" y1="4.5" x2="-0.5" y2="28.2" x3="-4.2" y3="16.35" textsize="3.5" layer="47" dtype="vertical"/>
+<dimension x1="3.3" y1="0" x2="3.3" y2="32.7" x3="-12.3" y3="16.35" textsize="3.5" layer="47" dtype="vertical"/>
+<dimension x1="4.35" y1="28.7" x2="16.05" y2="28.7" x3="10.2" y3="38.1" textsize="3.5" layer="47" dtype="horizontal"/>
 <text x="-5.6" y="-6.1" size="1.778" layer="46">1mm DIA. ROUTER PATH</text>
 <wire x1="10.2" y1="19.708" x2="10.2" y2="18.692" width="0.1016" layer="145"/>
@@
 </class>
 </classes>
-<designrules>
+<designrules name="default">
 <description language="de">&lt;b&gt;EAGLE Design Rules&lt;/b&gt;
 &lt;p&gt;
@@
 <attribute name="VALUE" x="12.3505" y="22.795" size="0.4064" layer="28" rot="MR270"/>
 </element>
-<element name="U$15" library="LITTLEBITS" package="LB_CREDITS_V2" value="LB_CREDITS_V2" x="-0.8" y="-22.25"/>
-<element name="U$16" library="SparkFun_NEW" package="OSHW-LOGO-L" value="OSHW-LOGOL" x="-21.2" y="-18.31"/>
+<element name="U$16" library="SparkFun_NEW" package="OSHW-LOGO-L" value="OSHW-LOGOL" x="-33.35" y="-60.91"/>
 <element name="O6BSM1" library="bitSnap" package="BITSNAP_V03_MALE" value="BITSNAP_V03_MALE" x="16.65" y="32.7" rot="R180"/>
 <element name="O6BSF1" library="bitSnap" package="BITSNAP_V03_FEMALE" value="BITSNAP_V03_FEMALE" x="3.75" y="0"/>
@@
 <attribute name="LB_PN" value="?" x="13.7" y="21.3" size="1.778" layer="28" rot="MR90" display="off"/>
 <attribute name="V_OPERATION" value="5V" x="13.7" y="21.3" size="1.778" layer="28" rot="MR90" display="off"/>
-<attribute name="IEC_ESD_PROT" value="+/-18kV" x="13.7" y="21.3" size="1.778" layer="28" rot="MR90" display="off"/>
 <attribute name="V_CLAMP" value="?" x="13.7" y="21.3" size="1.778" layer="28" rot="MR90" display="off"/>
 <attribute name="NAME" x="14.416" y="20.211" size="0.4064" layer="26" rot="MR90"/>
 <attribute name="VALUE" x="12.703" y="18.934" size="0.4064" layer="28" rot="MR90"/>
+<attribute name="MPN" value="ESD9B5.0ST5G" x="13.7" y="21.3" size="1.778" layer="28" rot="MR90" display="off"/>
+<attribute name="IEC_ESD_PROT0" value="+/-18kV" x="13.7" y="21.3" size="1.778" layer="28" rot="MR90" display="off"/>
 </element>
 <element name="O6C1" library="LITTLEBITS" package="CAP-0603" value="0.1 uF" x="6.75" y="21.35" smashed="yes" rot="MR270">
@@
 <attribute name="VALUE" x="5.643" y="19.866" size="0.4064" layer="28" font="vector" rot="MR180"/>
 </element>
-<element name="U$1" library="LITTLEBITS" package="FABDWG01-OHW" value="FRAME-LETTER-OHWOHW" x="-148.2" y="-76.45"/>
+<element name="U$1" library="LITTLEBITS" package="FABDWG01-OHW" value="FRAME-LETTER-OHWOHW" x="0" y="0"/>
+<element name="U$2" library="LITTLEBITS" package="OSHWCREDIT" value="OSHWCREDIT" x="-93.35" y="-64.55"/>
 </elements>
 <signals>
@@
 </board>
 </drawing>
+<compatibility>
+<note version="6.3" minversion="6.2.2" severity="warning">
+Since Version 6.2.2 text objects can contain more than one line,
+which will not be processed correctly with this version.
+</note>
+</compatibility>
 </eagle>

Commit message: Updated license text
Parts:
- moved U$16 8.25 mm to (-33.4, -69.2)
Changed lines of the file:
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@@
 <attribute name="VALUE" x="12.3505" y="22.795" size="0.4064" layer="28" rot="MR270"/>
 </element>
-<element name="U$16" library="SparkFun_NEW" package="OSHW-LOGO-L" value="OSHW-LOGOL" x="-33.35" y="-60.91"/>
+<element name="U$16" library="SparkFun_NEW" package="OSHW-LOGO-L" value="OSHW-LOGOL" x="-33.35" y="-69.16"/>
 <element name="O6BSM1" library="bitSnap" package="BITSNAP_V03_MALE" value="BITSNAP_V03_MALE" x="16.65" y="32.7" rot="R180"/>
 <element name="O6BSF1" library="bitSnap" package="BITSNAP_V03_FEMALE" value="BITSNAP_V03_FEMALE" x="3.75" y="0"/>
