File: OUTPUT/LB_Bit_o11_SERVO/LB_BIT_o11_servo-v03(rev4_4)/LB_BIT_o11_servo-v03(rev4_4).brd (EAGLE design)
At the start: 21.4 x 18.1 mm, 21 parts

Commit message: Updated licenses
Parts:
- moved U$1 162.9 mm to (0.00, 0.00)
- moved U$13 80.4 mm to (-69.4, -60.8)
- moved U$25 65.2 mm to (-77.3, -56.8)
Changed lines of the file:
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@@
 <?xml version="1.0" encoding="utf-8"?>
 <!DOCTYPE eagle SYSTEM "eagle.dtd">
-<eagle version="6.1">
+<eagle version="6.6.0">
 <drawing>
 <settings>
@@
 <layer number="54" name="bGND_GNDA" color="1" fill="9" visible="no" active="no"/>
 <layer number="56" name="wert" color="7" fill="1" visible="no" active="no"/>
+<layer number="57" name="tCAD" color="7" fill="1" visible="no" active="no"/>
 <layer number="91" name="Nets" color="2" fill="1" visible="no" active="no"/>
 <layer number="92" name="Busses" color="1" fill="1" visible="no" active="no"/>
@@
 <layer number="124" name="bTestmark" color="7" fill="1" visible="yes" active="yes"/>
 <layer number="125" name="_tNames" color="7" fill="1" visible="no" active="no"/>
+<layer number="150" name="Notes" color="7" fill="1" visible="yes" active="yes"/>
 <layer number="151" name="HeatSink" color="7" fill="1" visible="no" active="no"/>
 <layer number="152" name="_bDocu" color="7" fill="1" visible="yes" active="yes"/>
+<layer number="153" name="FabDoc1" color="6" fill="1" visible="no" active="no"/>
+<layer number="154" name="FabDoc2" color="2" fill="1" visible="no" active="no"/>
+<layer number="155" name="FabDoc3" color="7" fill="15" visible="no" active="no"/>
 <layer number="199" name="Contour" color="7" fill="1" visible="yes" active="yes"/>
 <layer number="200" name="200bmp" color="1" fill="10" visible="no" active="no"/>
@@
 <layer number="225" name="225bmp" color="26" fill="10" visible="no" active="no"/>
 <layer number="226" name="226bmp" color="27" fill="10" visible="no" active="no"/>
+<layer number="227" name="227bmp" color="7" fill="1" visible="yes" active="yes"/>
+<layer number="228" name="228bmp" color="7" fill="1" visible="yes" active="yes"/>
 <layer number="248" name="Housing" color="7" fill="1" visible="yes" active="yes"/>
 <layer number="249" name="Edge" color="7" fill="1" visible="yes" active="yes"/>
@@
 <wire x1="20.9" y1="22.1" x2="20.9" y2="4" width="1" layer="46"/>
 <wire x1="-0.5" y1="4" x2="-0.5" y2="22.1" width="1" layer="46"/>
-<dimension x1="3.8" y1="27" x2="16.6" y2="27" x3="10.2" y3="31.2" layer="47" dtype="horizontal"/>
-<dimension x1="20.4" y1="27" x2="0" y2="27" x3="10.2" y3="38.65" layer="47" dtype="horizontal"/>
-<dimension x1="-0.5" y1="4.5" x2="-0.5" y2="21.6" x3="-4.2" y3="13.05" layer="47" dtype="vertical"/>
-<dimension x1="3.3" y1="0" x2="3.3" y2="26.1" x3="-12.3" y3="13.05" layer="47" dtype="vertical"/>
-<dimension x1="4.35" y1="15.5" x2="16.05" y2="15.5" x3="10.2" y3="24.9" layer="47" dtype="horizontal"/>
+<dimension x1="3.8" y1="27" x2="16.6" y2="27" x3="10.2" y3="31.2" textsize="3.5" layer="47" dtype="horizontal"/>
+<dimension x1="20.4" y1="27" x2="0" y2="27" x3="10.2" y3="38.65" textsize="3.5" layer="47" dtype="horizontal"/>
+<dimension x1="-0.5" y1="4.5" x2="-0.5" y2="21.6" x3="-4.2" y3="13.05" textsize="3.5" layer="47" dtype="vertical"/>
+<dimension x1="3.3" y1="0" x2="3.3" y2="26.1" x3="-12.3" y3="13.05" textsize="3.5" layer="47" dtype="vertical"/>
+<dimension x1="4.35" y1="15.5" x2="16.05" y2="15.5" x3="10.2" y3="24.9" textsize="3.5" layer="47" dtype="horizontal"/>
 <text x="-6.5" y="-13.75" size="1.778" layer="46">1mm DIA. ROUTER PATH</text>
 <wire x1="0" y1="26.1" x2="20.4" y2="26.1" width="0" layer="49"/>
@@
 <wire x1="8.1" y1="13" x2="20.2" y2="13" width="0.2032" layer="42"/>
 <wire x1="13.8" y1="3.4" x2="16.2" y2="3.4" width="0.2032" layer="42"/>
-<text x="59.7" y="-44.8" size="1.778" layer="50">4</text>
-<text x="-7.4" y="-48.7" size="1.778" layer="50">Servo Motor Bit</text>
+<text x="56.35" y="-43.6" size="1.778" layer="50">4</text>
+<text x="-9.6" y="-47.5" size="1.778" layer="50">Servo Motor Bit</text>
 <wire x1="9.4" y1="7.408" x2="9.4" y2="6.392" width="0.1016" layer="145"/>
 <wire x1="8.892" y1="6.9" x2="9.908" y2="6.9" width="0.1016" layer="145"/>
@@
 </class>
 </classes>
-<designrules>
+<designrules name="default">
 <description language="de">&lt;b&gt;EAGLE Design Rules&lt;/b&gt;
 &lt;p&gt;
@@
 <attribute name="LB_PN" value="?" x="7.7" y="21.5" size="1.778" layer="28" rot="MR270" display="off"/>
 <attribute name="V_OPERATION" value="5V" x="7.7" y="21.5" size="1.778" layer="28" rot="MR270" display="off"/>
-<attribute name="IEC_ESD_PROT" value="+/-18kV" x="7.7" y="21.5" size="1.778" layer="28" rot="MR270" display="off"/>
 <attribute name="V_CLAMP" value="?" x="7.7" y="21.5" size="1.778" layer="28" rot="MR270" display="off"/>
 <attribute name="NAME" x="7.516" y="22.761" size="0.4064" layer="26" rot="MR90"/>
 <attribute name="VALUE" x="7.047" y="23.516" size="0.4064" layer="28" rot="MR270"/>
+<attribute name="MPN" value="ESD9B5.0ST5G" x="7.7" y="21.5" size="1.778" layer="28" rot="MR270" display="off"/>
+<attribute name="IEC_ESD_PROT0" value="+/-18kV" x="7.7" y="21.5" size="1.778" layer="28" rot="MR270" display="off"/>
 </element>
 <element name="O11R4" library="SparkFun" package="0603-RES" value="10k" x="10.2" y="21" smashed="yes" rot="MR180">
@@
 </element>
 <element name="U$26" library="ohw-logo" package="OSHW_FILLX150_NOTEXT" value="" x="15.8004" y="15.6587"/>
-<element name="U$13" library="LITTLEBITS" package="OSHWCREDIT" value="OSHWCREDIT" x="5.7" y="-32.1"/>
-<element name="U$25" library="LITTLEBITS" package="OSHW-LOGO-L" value="OSHW-LOGOL" x="-21" y="-23.85"/>
+<element name="U$13" library="LITTLEBITS" package="OSHWCREDIT" value="OSHWCREDIT" x="-69.4" y="-60.75"/>
+<element name="U$25" library="LITTLEBITS" package="OSHW-LOGO-L" value="OSHW-LOGOL" x="-77.3" y="-56.8"/>
 <element name="O11C4" library="SparkFun" package="0603-CAP" value="27p" x="18" y="10.2" smashed="yes" rot="MR90">
 <attribute name="NAME" x="18.762" y="9.311" size="0.4064" layer="26" font="vector" rot="MR90"/>
@@
 <attribute name="MFG" value="TXC" x="15.2" y="9.2" size="1.778" layer="28" rot="MR90" display="off"/>
 </element>
-<element name="U$1" library="LITTLEBITS" package="FABDWG01-OHW" value="FRAME-LETTER-OHWOHW" x="-144.05" y="-76"/>
+<element name="U$1" library="LITTLEBITS" package="FABDWG01-OHW" value="FRAME-LETTER-OHWOHW" x="0" y="0"/>
 </elements>
 <signals>
@@
 </board>
 </drawing>
+<compatibility>
+<note version="6.3" minversion="6.2.2" severity="warning">
+Since Version 6.2.2 text objects can contain more than one line,
+which will not be processed correctly with this version.
+</note>
+</compatibility>
 </eagle>

Commit message: Updated license text
Parts:
- moved U$25 49.5 mm to (-29.3, -68.8)
- moved U$13 21.9 mm to (-91.2, -63.5)
Changed lines of the file:
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@@
 </element>
 <element name="U$26" library="ohw-logo" package="OSHW_FILLX150_NOTEXT" value="" x="15.8004" y="15.6587"/>
-<element name="U$13" library="LITTLEBITS" package="OSHWCREDIT" value="OSHWCREDIT" x="-69.4" y="-60.75"/>
-<element name="U$25" library="LITTLEBITS" package="OSHW-LOGO-L" value="OSHW-LOGOL" x="-77.3" y="-56.8"/>
+<element name="U$13" library="LITTLEBITS" package="OSHWCREDIT" value="OSHWCREDIT" x="-91.15" y="-63.45"/>
+<element name="U$25" library="LITTLEBITS" package="OSHW-LOGO-L" value="OSHW-LOGOL" x="-29.3" y="-68.75"/>
 <element name="O11C4" library="SparkFun" package="0603-CAP" value="27p" x="18" y="10.2" smashed="yes" rot="MR90">
 <attribute name="NAME" x="18.762" y="9.311" size="0.4064" layer="26" font="vector" rot="MR90"/>
