File: POWER/LB_BIT_p3_USBPOWER/LB_BIT_p3_USBPOWER-v03(rev1)/LB_BIT_p3_USBPOWER-v03(rev1).brd (EAGLE design)
At the start: 21.4 x 16 mm, 10 parts, among them P3BSF1 BITSNAP_V03_FEMALE, P3C1 0.1uF, P3D1 Red, P3R1 220, P3X1 USB-MICROB-AUK_TH

Commit message: Updated licenses
Parts:
- removed U$17: FRAME-LETTER-OHWOHW, LITTLEBITS:FABDWG01-OHW
- added U$1: OSHWCREDIT, LITTLEBITS:OSHWCREDIT
- U$2: value LB_CREDITS_V2 -> FRAME-LETTER-OHWOHW; device LITTLEBITS:LB_CREDITS_V2 -> LITTLEBITS:FABDWG01-OHW
- moved U$2 43.8 mm to (-16.3, 9.65)
- moved U$3 22.3 mm to (-52.3, -48.0)
Changed lines of the file:
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@@
 <?xml version="1.0" encoding="utf-8"?>
 <!DOCTYPE eagle SYSTEM "eagle.dtd">
-<eagle version="6.1">
+<eagle version="6.6.0">
 <drawing>
 <settings>
@@
 <layer number="54" name="bGND_GNDA" color="1" fill="9" visible="no" active="no"/>
 <layer number="56" name="wert" color="7" fill="1" visible="yes" active="yes"/>
+<layer number="57" name="tCAD" color="7" fill="1" visible="no" active="no"/>
 <layer number="91" name="Nets" color="2" fill="1" visible="no" active="no"/>
 <layer number="92" name="Busses" color="1" fill="1" visible="no" active="no"/>
@@
 <layer number="145" name="DrillLegend_01-16" color="2" fill="9" visible="yes" active="yes"/>
 <layer number="146" name="DrillLegend_01-20" color="3" fill="9" visible="yes" active="yes"/>
+<layer number="150" name="Notes" color="7" fill="1" visible="yes" active="yes"/>
 <layer number="151" name="HeatSink" color="7" fill="1" visible="yes" active="yes"/>
 <layer number="152" name="_bDocu" color="7" fill="1" visible="yes" active="yes"/>
+<layer number="153" name="FabDoc1" color="6" fill="1" visible="no" active="no"/>
+<layer number="154" name="FabDoc2" color="2" fill="1" visible="no" active="no"/>
+<layer number="155" name="FabDoc3" color="7" fill="15" visible="no" active="no"/>
 <layer number="199" name="Contour" color="7" fill="1" visible="yes" active="yes"/>
 <layer number="200" name="200bmp" color="1" fill="10" visible="no" active="no"/>
@@
 <layer number="225" name="225bmp" color="26" fill="10" visible="yes" active="yes"/>
 <layer number="226" name="226bmp" color="27" fill="10" visible="yes" active="yes"/>
+<layer number="227" name="227bmp" color="7" fill="1" visible="yes" active="yes"/>
+<layer number="228" name="228bmp" color="7" fill="1" visible="yes" active="yes"/>
 <layer number="248" name="Housing" color="7" fill="1" visible="yes" active="yes"/>
 <layer number="249" name="Edge" color="7" fill="1" visible="yes" active="yes"/>
@@
 <wire x1="-16.9" y1="29.5" x2="4.5" y2="29.5" width="1" layer="46"/>
 <wire x1="4.5" y1="29.5" x2="4.5" y2="13.5" width="1" layer="46"/>
-<dimension x1="0.2" y1="9" x2="-12.6" y2="9" x3="-6.2" y3="-2.2" layer="47" dtype="horizontal"/>
-<dimension x1="-16.4" y1="13.5" x2="4" y2="13.5" x3="-6.2" y3="-9.65" layer="47" dtype="horizontal"/>
-<dimension x1="4.5" y1="29" x2="4.5" y2="14" x3="13.15" y3="21.5" layer="47" dtype="vertical"/>
-<dimension x1="4.5" y1="29" x2="0.7" y2="9.5" x3="21.3" y3="19.25" layer="47" dtype="vertical"/>
-<dimension x1="-0.35" y1="13.5" x2="-12.05" y2="13.5" x3="-6.2" y3="4.1" layer="47" dtype="horizontal"/>
+<dimension x1="0.2" y1="9" x2="-12.6" y2="9" x3="-6.2" y3="-2.2" textsize="3.5" layer="47" dtype="horizontal"/>
+<dimension x1="-16.4" y1="13.5" x2="4" y2="13.5" x3="-6.2" y3="-9.65" textsize="3.5" layer="47" dtype="horizontal"/>
+<dimension x1="4.5" y1="29" x2="4.5" y2="14" x3="13.15" y3="21.5" textsize="3.5" layer="47" dtype="vertical"/>
+<dimension x1="4.5" y1="29" x2="0.7" y2="9.5" x3="21.3" y3="19.25" textsize="3.5" layer="47" dtype="vertical"/>
+<dimension x1="-0.35" y1="13.5" x2="-12.05" y2="13.5" x3="-6.2" y3="4.1" textsize="3.5" layer="47" dtype="horizontal"/>
 <wire x1="-3.4154" y1="24.8855" x2="-2.3994" y2="23.8695" width="0.1016" layer="145"/>
 <wire x1="-2.3994" y1="24.8855" x2="-3.4154" y2="23.8695" width="0.1016" layer="145"/>
@@
 <wire x1="0.542" y1="22.35" x2="1.05" y2="22.858" width="0.1016" layer="146"/>
 <text x="-22.5" y="-16.35" size="1.778" layer="46">1mm DIA. ROUTER PATH</text>
-<text x="-30" y="-60.85" size="1.778" layer="50">p3 USB POWER BIT PCB</text>
-<text x="38" y="-56.85" size="1.778" layer="50">1</text>
+<text x="-27.65" y="-38.45" size="1.778" layer="50">p3 USB POWER BIT PCB</text>
+<text x="39.7" y="-34.1" size="1.778" layer="50">1</text>
 <text x="2.2" y="28.3" size="1.3" layer="21" font="vector" rot="SR270">p3 usb power</text>
 </plain>
@@
 </class>
 </classes>
-<designrules>
+<designrules name="default">
 <description language="en">&lt;b&gt;EAGLE Design Rules&lt;/b&gt;
 &lt;p&gt;
@@
 </element>
 <element name="U$4" library="ohw-logo" package="OSHW_FILLX150_NOTEXT" value="" x="-0.6285" y="23.1546"/>
-<element name="U$2" library="LITTLEBITS" package="LB_CREDITS_V2" value="LB_CREDITS_V2" x="-18.35" y="-34.15"/>
-<element name="U$3" library="SparkFun_NEW" package="OSHW-LOGO-L" value="OSHW-LOGOL" x="-38.75" y="-30.21"/>
+<element name="U$3" library="SparkFun_NEW" package="OSHW-LOGO-L" value="OSHW-LOGOL" x="-52.3" y="-47.96"/>
 <element name="P3BSF1" library="bitSnap" package="BITSNAP_V03_FEMALE" value="BITSNAP_V03_FEMALE" x="-12.65" y="9.5"/>
 <element name="U$15" library="LITTLEBITS" package="LB_PWR_LEGS" value="" x="-16.4" y="17.8"/>
-<element name="U$17" library="LITTLEBITS" package="FABDWG01-OHW" value="FRAME-LETTER-OHWOHW" x="-172.7" y="-88.55"/>
+<element name="U$1" library="LITTLEBITS" package="OSHWCREDIT" value="OSHWCREDIT" x="-108.05" y="-52.85"/>
+<element name="U$2" library="LITTLEBITS" package="FABDWG01-OHW" value="FRAME-LETTER-OHWOHW" x="-16.3" y="9.65"/>
 </elements>
 <signals>
@@
 </board>
 </drawing>
+<compatibility>
+<note version="6.3" minversion="6.2.2" severity="warning">
+Since Version 6.2.2 text objects can contain more than one line,
+which will not be processed correctly with this version.
+</note>
+</compatibility>
 </eagle>

Commit message: Updated license text
Parts:
- moved U$3 11.0 mm to (-49.4, -58.6)
Changed lines of the file:
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@@
 </element>
 <element name="U$4" library="ohw-logo" package="OSHW_FILLX150_NOTEXT" value="" x="-0.6285" y="23.1546"/>
-<element name="U$3" library="SparkFun_NEW" package="OSHW-LOGO-L" value="OSHW-LOGOL" x="-52.3" y="-47.96"/>
+<element name="U$3" library="SparkFun_NEW" package="OSHW-LOGO-L" value="OSHW-LOGOL" x="-49.4" y="-58.61"/>
 <element name="P3BSF1" library="bitSnap" package="BITSNAP_V03_FEMALE" value="BITSNAP_V03_FEMALE" x="-12.65" y="9.5"/>
 <element name="U$15" library="LITTLEBITS" package="LB_PWR_LEGS" value="" x="-16.4" y="17.8"/>
