File: WIRE/LB_BIT_w10_INVERTER/LB_BIT_w10_INVERTER_v03(rev1)/LB_w10_INVERTER_v03(rev1).brd (EAGLE design)
At the start: 21.4 x 11.5 mm, 9 parts

Commit message: Updated licenses
Parts:
- U$3: value LB_CREDITS_V2 -> OSHWCREDIT; device LITTLEBITS:LB_CREDITS_V2 -> LITTLEBITS:OSHWCREDIT
- moved U$1 181.4 mm to (0.00, 0.00)
- moved U$3 101.5 mm to (-91.0, -64.7)
- moved U$4 49.6 mm to (-33.0, -59.9)
Changed lines of the file:
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@@
 <?xml version="1.0" encoding="utf-8"?>
 <!DOCTYPE eagle SYSTEM "eagle.dtd">
-<eagle version="6.1">
+<eagle version="6.6.0">
 <drawing>
 <settings>
@@
 <layer number="54" name="bGND_GNDA" color="1" fill="9" visible="no" active="no"/>
 <layer number="56" name="wert" color="7" fill="1" visible="no" active="no"/>
+<layer number="57" name="tCAD" color="7" fill="1" visible="no" active="no"/>
 <layer number="91" name="Nets" color="2" fill="1" visible="no" active="no"/>
 <layer number="92" name="Busses" color="1" fill="1" visible="no" active="no"/>
@@
 <layer number="124" name="bTestmark" color="7" fill="1" visible="yes" active="yes"/>
 <layer number="125" name="_tNames" color="7" fill="1" visible="no" active="no"/>
+<layer number="150" name="Notes" color="7" fill="1" visible="yes" active="yes"/>
 <layer number="151" name="HeatSink" color="7" fill="1" visible="no" active="no"/>
 <layer number="152" name="_bDocu" color="7" fill="1" visible="yes" active="yes"/>
+<layer number="153" name="FabDoc1" color="6" fill="1" visible="no" active="no"/>
+<layer number="154" name="FabDoc2" color="2" fill="1" visible="no" active="no"/>
+<layer number="155" name="FabDoc3" color="7" fill="15" visible="no" active="no"/>
 <layer number="199" name="Contour" color="7" fill="1" visible="yes" active="yes"/>
 <layer number="200" name="200bmp" color="1" fill="10" visible="no" active="no"/>
@@
 <layer number="225" name="225bmp" color="26" fill="10" visible="no" active="no"/>
 <layer number="226" name="226bmp" color="27" fill="10" visible="no" active="no"/>
+<layer number="227" name="227bmp" color="7" fill="1" visible="yes" active="yes"/>
+<layer number="228" name="228bmp" color="7" fill="1" visible="yes" active="yes"/>
 <layer number="248" name="Housing" color="7" fill="1" visible="yes" active="yes"/>
 <layer number="249" name="Edge" color="7" fill="1" visible="yes" active="yes"/>
@@
 <wire x1="20.9" y1="15.5" x2="20.9" y2="4" width="1" layer="46"/>
 <wire x1="20.9" y1="4" x2="20.4" y2="4" width="1" layer="46"/>
-<dimension x1="3.8" y1="20" x2="16.6" y2="20" x3="10.2" y3="31.2" layer="47" dtype="horizontal"/>
-<dimension x1="20.4" y1="15.5" x2="0" y2="15.5" x3="10.2" y3="38.65" layer="47" dtype="horizontal"/>
-<dimension x1="-0.5" y1="4.5" x2="-0.5" y2="15" x3="-4.2" y3="9.75" layer="47" dtype="vertical"/>
-<dimension x1="3.3" y1="0" x2="3.3" y2="19.5" x3="-12.3" y3="9.75" layer="47" dtype="vertical"/>
-<dimension x1="4.35" y1="15.5" x2="16.05" y2="15.5" x3="10.2" y3="24.9" layer="47" dtype="horizontal"/>
+<dimension x1="3.8" y1="20" x2="16.6" y2="20" x3="10.2" y3="31.2" textsize="3.5" layer="47" dtype="horizontal"/>
+<dimension x1="20.4" y1="15.5" x2="0" y2="15.5" x3="10.2" y3="38.65" textsize="3.5" layer="47" dtype="horizontal"/>
+<dimension x1="-0.5" y1="4.5" x2="-0.5" y2="15" x3="-4.2" y3="9.75" textsize="3.5" layer="47" dtype="vertical"/>
+<dimension x1="3.3" y1="0" x2="3.3" y2="19.5" x3="-12.3" y3="9.75" textsize="3.5" layer="47" dtype="vertical"/>
+<dimension x1="4.35" y1="15.5" x2="16.05" y2="15.5" x3="10.2" y3="24.9" textsize="3.5" layer="47" dtype="horizontal"/>
 <wire x1="14.1" y1="7.908" x2="14.1" y2="6.892" width="0.1016" layer="145"/>
 <wire x1="13.592" y1="7.4" x2="14.608" y2="7.4" width="0.1016" layer="145"/>
@@
 </class>
 </classes>
-<designrules>
+<designrules name="default">
 <description language="en">&lt;b&gt;EAGLE Design Rules&lt;/b&gt;
 &lt;p&gt;
@@
 <attribute name="VALUE" x="13.212" y="10.691" size="0.4064" layer="27" font="vector" rot="R270"/>
 </element>
-<element name="U$3" library="LITTLEBITS" package="LB_CREDITS_V2" value="LB_CREDITS_V2" x="-0.6" y="-18.48"/>
-<element name="U$4" library="SparkFun_NEW" package="OSHW-LOGO-L" value="OSHW-LOGOL" x="-13.25" y="-14.39"/>
+<element name="U$4" library="SparkFun_NEW" package="OSHW-LOGO-L" value="OSHW-LOGOL" x="-32.95" y="-59.89"/>
 <element name="U$2" library="ohw-logo" package="OSHW_FILLX150_NOTEXT" value="" x="15.7992375" y="9.260871875"/>
 <element name="W10BSM1" library="bitSnap" package="BITSNAP_V03_MALE" value="BITSNAP_V03_MALE" x="16.65" y="19.5" rot="R180"/>
 <element name="W10BSF1" library="bitSnap" package="BITSNAP_V03_FEMALE" value="BITSNAP_V03_FEMALE" x="3.75" y="0"/>
-<element name="U$1" library="LITTLEBITS" package="FABDWG01-OHW" value="FRAME-LETTER-OHWOHW" x="-166.3" y="-72.55"/>
+<element name="U$1" library="LITTLEBITS" package="FABDWG01-OHW" value="FRAME-LETTER-OHWOHW" x="0" y="0"/>
+<element name="U$3" library="LITTLEBITS" package="OSHWCREDIT" value="OSHWCREDIT" x="-91" y="-64.65"/>
 </elements>
 <signals>
@@
 </board>
 </drawing>
+<compatibility>
+<note version="6.3" minversion="6.2.2" severity="warning">
+Since Version 6.2.2 text objects can contain more than one line,
+which will not be processed correctly with this version.
+</note>
+</compatibility>
 </eagle>

Commit message: Updated license text
Parts:
- moved U$4 9.50 mm to (-30.8, -69.1)
Changed lines of the file:
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@@
 <attribute name="VALUE" x="13.212" y="10.691" size="0.4064" layer="27" font="vector" rot="R270"/>
 </element>
-<element name="U$4" library="SparkFun_NEW" package="OSHW-LOGO-L" value="OSHW-LOGOL" x="-32.95" y="-59.89"/>
+<element name="U$4" library="SparkFun_NEW" package="OSHW-LOGO-L" value="OSHW-LOGOL" x="-30.8" y="-69.14"/>
 <element name="U$2" library="ohw-logo" package="OSHW_FILLX150_NOTEXT" value="" x="15.7992375" y="9.260871875"/>
 <element name="W10BSM1" library="bitSnap" package="BITSNAP_V03_MALE" value="BITSNAP_V03_MALE" x="16.65" y="19.5" rot="R180"/>
