File: WIRE/LB_BIT_w1_WIRE/LB_BIT_w1_WIRE-v03(rev2)/LB_BIT_w1_Wire_South-v03(rev2)/LB_w1_Wire_South-v03(rev2).sch (EAGLE design)
At the start: 5 parts

Commit message: Updated licenses
Parts:
- removed U$4: LB_CREDITS, LITTLEBITS:LB_CREDITS
- added U$1: OSHWCREDIT, LITTLEBITS:OSHWCREDIT
Other:
- note added: "in collaboration with Chris Taylor from SparkFun"
Changed lines of the file:
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@@
 <?xml version="1.0" encoding="utf-8"?>
 <!DOCTYPE eagle SYSTEM "eagle.dtd">
-<eagle version="6.4">
+<eagle version="6.6.0">
 <drawing>
 <settings>
@@
 <layer number="54" name="bGND_GNDA" color="1" fill="9" visible="no" active="no"/>
 <layer number="56" name="wert" color="7" fill="1" visible="no" active="no"/>
+<layer number="57" name="tCAD" color="7" fill="1" visible="no" active="no"/>
 <layer number="91" name="Nets" color="2" fill="1" visible="yes" active="yes"/>
 <layer number="92" name="Busses" color="1" fill="1" visible="yes" active="yes"/>
@@
 <layer number="145" name="DrillLegend_01-16" color="2" fill="9" visible="yes" active="yes"/>
 <layer number="146" name="DrillLegend_01-20" color="3" fill="9" visible="yes" active="yes"/>
+<layer number="150" name="Notes" color="7" fill="1" visible="yes" active="yes"/>
 <layer number="151" name="HeatSink" color="7" fill="1" visible="yes" active="yes"/>
 <layer number="152" name="_bDocu" color="7" fill="1" visible="yes" active="yes"/>
+<layer number="153" name="FabDoc1" color="6" fill="1" visible="no" active="no"/>
+<layer number="154" name="FabDoc2" color="2" fill="1" visible="no" active="no"/>
+<layer number="155" name="FabDoc3" color="7" fill="15" visible="no" active="no"/>
 <layer number="199" name="Contour" color="7" fill="1" visible="yes" active="yes"/>
 <layer number="200" name="200bmp" color="1" fill="10" visible="no" active="no"/>
@@
 <layer number="225" name="225bmp" color="26" fill="10" visible="no" active="yes"/>
 <layer number="226" name="226bmp" color="27" fill="10" visible="no" active="yes"/>
+<layer number="227" name="227bmp" color="7" fill="1" visible="yes" active="yes"/>
+<layer number="228" name="228bmp" color="7" fill="1" visible="yes" active="yes"/>
 <layer number="248" name="Housing" color="7" fill="1" visible="yes" active="yes"/>
 <layer number="249" name="Edge" color="7" fill="1" visible="yes" active="yes"/>
@@
 <part name="W1JP1" library="SparkFun" deviceset="M03" device="SMD"/>
 <part name="U$3" library="SparkFun" deviceset="OSHW-LOGO" device="L"/>
-<part name="U$4" library="LITTLEBITS" deviceset="LB_CREDITS" device=""/>
 <part name="W1BSF1" library="bitSnap" deviceset="BITSNAP_V03_FEMALE" device=""/>
+<part name="U$1" library="LITTLEBITS" deviceset="OSHWCREDIT" device=""/>
 </parts>
 <sheets>
@@
 <plain>
 <text x="241.3" y="12.7" size="2.54" layer="91">2</text>
+<text x="50.8" y="15.24" size="1.778" layer="97">in collaboration with Chris Taylor from SparkFun</text>
 </plain>
 <instances>
@@
 <instance part="W1JP1" gate="G$1" x="109.22" y="106.68" rot="MR180"/>
 <instance part="U$3" gate="G$1" x="134.62" y="10.16"/>
-<instance part="U$4" gate="G$1" x="43.18" y="12.7"/>
 <instance part="W1BSF1" gate="G$1" x="124.46" y="101.6"/>
+<instance part="U$1" gate="G$1" x="48.26" y="17.78"/>
 </instances>
 <busses>
@@
 </schematic>
 </drawing>
+<compatibility>
+<note version="6.3" minversion="6.2.2" severity="warning">
+Since Version 6.2.2 text objects can contain more than one line,
+which will not be processed correctly with this version.
+</note>
+</compatibility>
 </eagle>

Commit message: Updated license text
Changed lines of the file:
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@@
 <plain>
 <text x="241.3" y="12.7" size="2.54" layer="91">2</text>
-<text x="50.8" y="15.24" size="1.778" layer="97">in collaboration with Chris Taylor from SparkFun</text>
+<text x="62.738" y="17.272" size="1.27" layer="97">in collaboration with Chris Taylor from SparkFun</text>
 </plain>
 <instances>
