File: WIRE/LB_BIT_w4_DOUBLE_AND/LB_w4_DOUBLEAND-v03(rev4)/LB-w4-DOUBLE_AND_v03(rev4).brd (EAGLE design)
At the start: 21.4 x 29.2 mm, 15 parts

Commit message: Updated licenses
Parts:
- removed U$17: LB_CREDITS_V2, LITTLEBITS:LB_CREDITS_V2
- added U$2: OSHWCREDIT, LITTLEBITS:OSHWCREDIT
- moved FRAME1 115.3 mm to (-0.03, 0.00)
- moved U$1 72.8 mm to (-39.3, -60.9)
Changed lines of the file:
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@@
 <?xml version="1.0" encoding="utf-8"?>
 <!DOCTYPE eagle SYSTEM "eagle.dtd">
-<eagle version="6.1">
+<eagle version="6.6.0">
 <drawing>
 <settings>
@@
 <layer number="54" name="bGND_GNDA" color="1" fill="9" visible="no" active="no"/>
 <layer number="56" name="wert" color="7" fill="1" visible="yes" active="yes"/>
+<layer number="57" name="tCAD" color="7" fill="1" visible="no" active="no"/>
 <layer number="91" name="Nets" color="2" fill="1" visible="no" active="no"/>
 <layer number="92" name="Busses" color="1" fill="1" visible="no" active="no"/>
@@
 <layer number="145" name="DrillLegend_01-16" color="2" fill="9" visible="yes" active="yes"/>
 <layer number="146" name="DrillLegend_01-20" color="3" fill="9" visible="yes" active="yes"/>
+<layer number="150" name="Notes" color="7" fill="1" visible="yes" active="yes"/>
 <layer number="151" name="HeatSink" color="7" fill="1" visible="yes" active="yes"/>
 <layer number="152" name="_bDocu" color="7" fill="1" visible="yes" active="yes"/>
+<layer number="153" name="FabDoc1" color="6" fill="1" visible="no" active="no"/>
+<layer number="154" name="FabDoc2" color="2" fill="1" visible="no" active="no"/>
+<layer number="155" name="FabDoc3" color="7" fill="15" visible="no" active="no"/>
 <layer number="199" name="Contour" color="7" fill="1" visible="yes" active="yes"/>
 <layer number="200" name="200bmp" color="1" fill="10" visible="no" active="no"/>
@@
 <layer number="225" name="225bmp" color="26" fill="10" visible="yes" active="yes"/>
 <layer number="226" name="226bmp" color="27" fill="10" visible="yes" active="yes"/>
+<layer number="227" name="227bmp" color="7" fill="1" visible="yes" active="yes"/>
+<layer number="228" name="228bmp" color="7" fill="1" visible="yes" active="yes"/>
 <layer number="248" name="Housing" color="7" fill="1" visible="yes" active="yes"/>
 <layer number="249" name="Edge" color="7" fill="1" visible="yes" active="yes"/>
@@
 <wire x1="4.5" y1="33.2" x2="4.5" y2="29.9" width="1" layer="46"/>
 <wire x1="4.5" y1="29.9" x2="6.2" y2="29.9" width="1" layer="46"/>
-<dimension x1="8.35" y1="0.1" x2="4.5" y2="32.7" x3="-37.7" y3="16.4" layer="47" dtype="vertical"/>
-<dimension x1="1.7" y1="13.3" x2="1.7" y2="26.1" x3="-24.95" y3="19.7" layer="47" dtype="vertical"/>
-<dimension x1="4.55" y1="4.6" x2="2.15" y2="0.1" x3="-30.35" y3="2.35" layer="47" dtype="vertical"/>
-<dimension x1="4.55" y1="9" x2="1.7" y2="13.3" x3="-0.65" y3="11.15" layer="47" dtype="vertical"/>
-<dimension x1="1.7" y1="26.1" x2="4.55" y2="30.4" x3="-10.2" y3="28.25" layer="47" dtype="vertical"/>
-<dimension x1="6.2" y1="25.55" x2="6.2" y2="13.85" x3="-17" y3="19.7" layer="47" dtype="vertical"/>
-<dimension x1="21.6" y1="-0.5" x2="8.8" y2="-0.5" x3="15.2" y3="-11.7" layer="47" dtype="horizontal"/>
-<dimension x1="5" y1="4" x2="25.4" y2="4" x3="15.2" y3="-19.15" layer="47" dtype="horizontal"/>
-<dimension x1="21.05" y1="4" x2="9.35" y2="4" x3="15.2" y3="-5.4" layer="47" dtype="horizontal"/>
-<dimension x1="-5.7" y1="4.6" x2="-5.4" y2="0.1" x3="-7.85" y3="2.35" layer="47" dtype="vertical"/>
+<dimension x1="8.35" y1="0.1" x2="4.5" y2="32.7" x3="-37.7" y3="16.4" textsize="3.5" layer="47" dtype="vertical"/>
+<dimension x1="1.7" y1="13.3" x2="1.7" y2="26.1" x3="-24.95" y3="19.7" textsize="3.5" layer="47" dtype="vertical"/>
+<dimension x1="4.55" y1="4.6" x2="2.15" y2="0.1" x3="-30.35" y3="2.35" textsize="3.5" layer="47" dtype="vertical"/>
+<dimension x1="4.55" y1="9" x2="1.7" y2="13.3" x3="-0.65" y3="11.15" textsize="3.5" layer="47" dtype="vertical"/>
+<dimension x1="1.7" y1="26.1" x2="4.55" y2="30.4" x3="-10.2" y3="28.25" textsize="3.5" layer="47" dtype="vertical"/>
+<dimension x1="6.2" y1="25.55" x2="6.2" y2="13.85" x3="-17" y3="19.7" textsize="3.5" layer="47" dtype="vertical"/>
+<dimension x1="21.6" y1="-0.5" x2="8.8" y2="-0.5" x3="15.2" y3="-11.7" textsize="3.5" layer="47" dtype="horizontal"/>
+<dimension x1="5" y1="4" x2="25.4" y2="4" x3="15.2" y3="-19.15" textsize="3.5" layer="47" dtype="horizontal"/>
+<dimension x1="21.05" y1="4" x2="9.35" y2="4" x3="15.2" y3="-5.4" textsize="3.5" layer="47" dtype="horizontal"/>
+<dimension x1="-5.7" y1="4.6" x2="-5.4" y2="0.1" x3="-7.85" y3="2.35" textsize="3.5" layer="47" dtype="vertical"/>
 <wire x1="6.7" y1="9.5" x2="6.2" y2="9" width="0" layer="20" curve="-90"/>
 <wire x1="24.2" y1="9" x2="23.7" y2="9.5" width="0" layer="20" curve="-90"/>
 <wire x1="6.2" y1="30.4" x2="6.7" y2="29.9" width="0" layer="20" curve="-90"/>
 <wire x1="23.7" y1="29.9" x2="24.2" y2="30.4" width="0" layer="20" curve="-90"/>
-<dimension x1="6.7" y1="30.7" x2="23.7" y2="30.7" x3="15.2" y3="35.85" layer="47" dtype="horizontal"/>
-<dimension x1="2.2" y1="26.6" x2="28.2" y2="26.6" x3="15.2" y3="42.1" layer="47" dtype="horizontal"/>
+<dimension x1="6.7" y1="30.7" x2="23.7" y2="30.7" x3="15.2" y3="35.85" textsize="3.5" layer="47" dtype="horizontal"/>
+<dimension x1="2.2" y1="26.6" x2="28.2" y2="26.6" x3="15.2" y3="42.1" textsize="3.5" layer="47" dtype="horizontal"/>
 <text x="-2.65" y="52" size="1.778" layer="46">1mm DIA. ROUTER PATH</text>
-<text x="48.2" y="-46.25" size="1.778" layer="50">w4 DOUBLE AND BIT PCB</text>
+<text x="-11" y="-47.65" size="1.778" layer="50">w4 DOUBLE AND BIT PCB</text>
 <text x="114.7" y="-42.25" size="1.778" layer="50">4</text>
 <wire x1="17.1" y1="24.108" x2="17.1" y2="23.092" width="0.1016" layer="145"/>
@@
 </class>
 </classes>
-<designrules>
+<designrules name="default">
 <description language="en">&lt;b&gt;EAGLE Design Rules&lt;/b&gt;
 &lt;p&gt;
@@
 <attribute name="VALUE" x="10.453" y="19.966" size="0.3048" layer="27" rot="R270"/>
 </element>
-<element name="U$1" library="SparkFun_NEW" package="OSHW-LOGO-L" value="OSHW-LOGOL" x="33.08" y="-68.46"/>
+<element name="U$1" library="SparkFun_NEW" package="OSHW-LOGO-L" value="OSHW-LOGOL" x="-39.32" y="-60.86"/>
 <element name="W4BSM1" library="bitSnap" package="BITSNAP_V03_MALE" value="BITSNAP_V03_MALE" x="2.2" y="26.15" rot="R270"/>
 <element name="W4BSF1" library="bitSnap" package="BITSNAP_V03_FEMALE" value="BITSNAP_V03_FEMALE" x="8.75" y="0"/>
 <element name="W4BSM2" library="bitSnap" package="BITSNAP_V03_MALE" value="BITSNAP_V03_MALE" x="28.2" y="13.25" rot="R90"/>
 <element name="U$3" library="bitSnap" package="AND/OR_OVERLAY" value="" x="4.75" y="-3.05"/>
-<element name="U$17" library="LITTLEBITS" package="LB_CREDITS_V2" value="LB_CREDITS_V2" x="-9.42" y="-62.9"/>
 <element name="W4U2" library="LITTLEBITS" package="SC70-6" value="SCHMITT_TRIGGER_NON_INVERTING NC7WZ17" x="15.2" y="22.76" smashed="yes" rot="R180">
 <attribute name="LB_PN" value="" x="15.2" y="22.76" size="1.778" layer="27" rot="R180" display="off"/>
@@
 <attribute name="VOLTAGE" value="" x="18.7" y="22.7" size="1.778" layer="27" rot="R90" display="off"/>
 </element>
-<element name="FRAME1" library="LITTLEBITS" package="FABDWG01-OHW" value="FRAME-LETTER-OHWOHW" x="-88.4789" y="-73.95"/>
+<element name="FRAME1" library="LITTLEBITS" package="FABDWG01-OHW" value="FRAME-LETTER-OHWOHW" x="-0.0289" y="0"/>
+<element name="U$2" library="LITTLEBITS" package="OSHWCREDIT" value="OSHWCREDIT" x="-92.15" y="-66.1"/>
 </elements>
 <signals>
@@
 <contactref element="W4C1" pad="2"/>
 <via x="17.1" y="23.6" extent="1-16" drill="0.6"/>
-<wire x1="15.2" y1="23.585" x2="15.2" y2="24.45" width="0.4064" layer="1"/>
+<wire x1="15.2" y1="23.66" x2="15.2" y2="24.45" width="0.4064" layer="1"/>
 <wire x1="15.2" y1="24.45" x2="14.95" y2="24.7" width="0.4064" layer="1"/>
 <wire x1="14.95" y1="24.7" x2="14.7" y2="24.7" width="0.4064" layer="1"/>
@@
 <wire x1="16.15" y1="16.65" x2="16.15" y2="17.95" width="0.6" layer="1"/>
 <wire x1="18.7" y1="21.85" x2="18.7" y2="19.1" width="0.6" layer="1"/>
-<wire x1="15.2" y1="21.935" x2="15.2" y2="22.6" width="0.4" layer="1"/>
+<wire x1="15.2" y1="21.86" x2="15.2" y2="22.6" width="0.4" layer="1"/>
 <wire x1="15.2" y1="22.6" x2="15.35" y2="22.75" width="0.4" layer="1"/>
 <wire x1="15.35" y1="22.75" x2="16.25" y2="22.75" width="0.4" layer="1"/>
@@
 <via x="10.45" y="23.6" extent="1-16" drill="0.6"/>
 <wire x1="10.45" y1="23.6" x2="14.535" y2="23.6" width="0.4" layer="1"/>
-<wire x1="14.535" y1="23.6" x2="14.55" y2="23.585" width="0.2" layer="1"/>
+<wire x1="14.535" y1="23.6" x2="14.55" y2="23.66" width="0.2" layer="1"/>
 <wire x1="10.45" y1="23.6" x2="11.7" y2="23.6" width="0.4064" layer="1"/>
 <wire x1="11.7" y1="23.6" x2="11.7" y2="23.55" width="0.4064" layer="1"/>
@@
 <wire x1="20.1" y1="26" x2="15.9" y2="26" width="0.6" layer="1"/>
 <wire x1="15.9" y1="26" x2="15.85" y2="25.85" width="0.6" layer="1"/>
-<wire x1="15.85" y1="25.85" x2="15.85" y2="23.585" width="0.4" layer="1"/>
+<wire x1="15.85" y1="25.85" x2="15.85" y2="23.66" width="0.4" layer="1"/>
 <wire x1="23.3813" y1="19.7213" x2="23.35" y2="19.69" width="0.2" layer="1"/>
 <wire x1="15.9" y1="26" x2="16.05" y2="26" width="0" layer="19" extent="1-1"/>
@@
 <contactref element="W4U2" pad="6"/>
 <contactref element="W4U1" pad="1"/>
-<wire x1="15.85" y1="21.935" x2="15.85" y2="21.15" width="0.4" layer="1"/>
+<wire x1="15.85" y1="21.86" x2="15.85" y2="21.15" width="0.4" layer="1"/>
 <wire x1="15.85" y1="21.15" x2="16.15" y2="20.85" width="0.4" layer="1"/>
 <wire x1="16.15" y1="20.85" x2="16.15" y2="19.24" width="0.4" layer="1"/>
@@
 <contactref element="W4U2" pad="4"/>
 <contactref element="W4U1" pad="2"/>
-<wire x1="14.55" y1="21.935" x2="14.55" y2="20.9" width="0.4" layer="1"/>
+<wire x1="14.55" y1="21.86" x2="14.55" y2="20.9" width="0.4" layer="1"/>
 <wire x1="14.55" y1="20.9" x2="15.2" y2="20.25" width="0.4" layer="1"/>
 <wire x1="15.2" y1="20.25" x2="15.2" y2="19.2342" width="0.4" layer="1"/>
@@
 </board>
 </drawing>
+<compatibility>
+<note version="6.3" minversion="6.2.2" severity="warning">
+Since Version 6.2.2 text objects can contain more than one line,
+which will not be processed correctly with this version.
+</note>
+</compatibility>
 </eagle>

Commit message: Updated license text
Parts:
- moved U$1 11.4 mm to (-33.2, -70.5)
Changed lines of the file:
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@@
 <attribute name="VALUE" x="10.453" y="19.966" size="0.3048" layer="27" rot="R270"/>
 </element>
-<element name="U$1" library="SparkFun_NEW" package="OSHW-LOGO-L" value="OSHW-LOGOL" x="-39.32" y="-60.86"/>
+<element name="U$1" library="SparkFun_NEW" package="OSHW-LOGO-L" value="OSHW-LOGOL" x="-33.22" y="-70.46"/>
 <element name="W4BSM1" library="bitSnap" package="BITSNAP_V03_MALE" value="BITSNAP_V03_MALE" x="2.2" y="26.15" rot="R270"/>
 <element name="W4BSF1" library="bitSnap" package="BITSNAP_V03_FEMALE" value="BITSNAP_V03_FEMALE" x="8.75" y="0"/>
