File: WIRE/LB_BIT_w6_ARDUINO/LB_BIT_w6_ARDUINO-v03(4-5)/LB_BIT_w6_ARDUINO-v03(4-5)OHW.sch (EAGLE design)
At the start: 75 parts

Commit message: Updated address and license.
Parts:
- removed U$68: OSHWCREDIT, LITTLEBITS:OSHWCREDIT
Changed lines of the file:
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@@
 <part name="P+23" library="LITTLEBITS" deviceset="VCC" device=""/>
 <part name="U$67" library="LITTLEBITS" deviceset="OSHWCREDIT" device=""/>
-<part name="U$68" library="LITTLEBITS" deviceset="OSHWCREDIT" device=""/>
 <part name="U$70" library="LITTLEBITS" deviceset="OSHW-LOGO" device="L"/>
 <part name="W6C28" library="LITTLEBITS" deviceset="CAP" device="CAP-0603" value="1000pF"/>
@@
 <text x="215.9" y="132.08" size="1.778" layer="91">RX</text>
 <text x="215.9" y="124.46" size="1.778" layer="91">TX</text>
-<text x="22.86" y="2.54" size="1.778" layer="97">Based on the Leonardo design by Arduino
+<text x="5.08" y="2.54" size="1.778" layer="97">Based on the Leonardo design by Arduino
 http://arduino.cc</text>
 </plain>
@@
 <instance part="P+22" gate="1" x="177.8" y="81.28" rot="MR180"/>
 <instance part="P+23" gate="1" x="185.42" y="81.28" rot="MR180"/>
-<instance part="U$67" gate="G$1" x="35.56" y="7.62"/>
+<instance part="U$67" gate="G$1" x="5.08" y="7.62"/>
 <instance part="W6C28" gate="G$1" x="220.98" y="157.48" rot="R90"/>
 <instance part="W6C29" gate="G$1" x="220.98" y="147.32" rot="R90"/>
@@
 <instance part="W6TVS4" gate="G$1" x="182.88" y="157.48"/>
 <instance part="W6TVS1" gate="G$1" x="53.34" y="134.62"/>
-<instance part="U$68" gate="G$1" x="35.56" y="10.16"/>
 <instance part="U$70" gate="G$1" x="132.08" y="12.7"/>
 <instance part="GND23" gate="1" x="124.46" y="91.44"/>

Commit message: Updated PDFs
Parts:
- added U$1: OSHWCREDIT, LITTLEBITS:OSHWCREDIT
Changed lines of the file:
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@@
 <part name="U$52" library="LITTLEBITS" deviceset="OSHW-LOGO" device="L"/>
 <part name="U$54" library="LITTLEBITS" deviceset="FRAME-LETTER-OHW" device="OHW"/>
+<part name="U$1" library="LITTLEBITS" deviceset="OSHWCREDIT" device=""/>
 </parts>
 <sheets>
@@
 <instance part="U$54" gate="G$1" x="0" y="0"/>
 <instance part="U$54" gate="G$2" x="147.32" y="0"/>
+<instance part="U$1" gate="G$1" x="22.86" y="12.7"/>
 </instances>
 <busses>

Commit message: Updated license text
Parts:
- removed U$1: OSHWCREDIT, LITTLEBITS:OSHWCREDIT
Changed lines of the file:
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@@
 <?xml version="1.0" encoding="utf-8"?>
 <!DOCTYPE eagle SYSTEM "eagle.dtd">
-<eagle version="6.5.0">
+<eagle version="6.6.0">
 <drawing>
 <settings>
@@
 <part name="U$52" library="LITTLEBITS" deviceset="OSHW-LOGO" device="L"/>
 <part name="U$54" library="LITTLEBITS" deviceset="FRAME-LETTER-OHW" device="OHW"/>
-<part name="U$1" library="LITTLEBITS" deviceset="OSHWCREDIT" device=""/>
 </parts>
 <sheets>
@@
 <instance part="P+22" gate="1" x="177.8" y="81.28" rot="MR180"/>
 <instance part="P+23" gate="1" x="185.42" y="81.28" rot="MR180"/>
-<instance part="U$67" gate="G$1" x="5.08" y="7.62"/>
+<instance part="U$67" gate="G$1" x="5.08" y="15.24"/>
 <instance part="W6C28" gate="G$1" x="220.98" y="157.48" rot="R90"/>
 <instance part="W6C29" gate="G$1" x="220.98" y="147.32" rot="R90"/>
@@
 <instance part="U$54" gate="G$1" x="0" y="0"/>
 <instance part="U$54" gate="G$2" x="147.32" y="0"/>
-<instance part="U$1" gate="G$1" x="22.86" y="12.7"/>
 </instances>
 <busses>
