File: WIRE/LB_BIT_w7_FORK/LB_BIT_w7_FORK-v03(rev1)/LB_BIT_w7_FORK-v03(rev1).brd (EAGLE design)
At the start: 74.2 x 11.5 mm, 9 parts

Commit message: Updated licenses
Parts:
- removed U$1: (no value), LITTLEBITS:OSHW-LOGO-L
- added U$2: OSHW-LOGOL, LITTLEBITS:OSHW-LOGO-L
- moved FRAME1 174.1 mm to (28.4, -5.85)
- moved U$12 25.8 mm to (-63.8, -71.8)
Changed lines of the file:
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@@
 <?xml version="1.0" encoding="utf-8"?>
 <!DOCTYPE eagle SYSTEM "eagle.dtd">
-<eagle version="6.1">
+<eagle version="6.6.0">
 <drawing>
 <settings>
@@
 <layer number="54" name="bGND_GNDA" color="7" fill="1" visible="yes" active="yes"/>
 <layer number="56" name="wert" color="7" fill="1" visible="yes" active="yes"/>
+<layer number="57" name="tCAD" color="7" fill="1" visible="no" active="no"/>
 <layer number="91" name="Nets" color="2" fill="1" visible="no" active="no"/>
 <layer number="92" name="Busses" color="1" fill="1" visible="no" active="no"/>
@@
 <layer number="145" name="DrillLegend_01-16" color="2" fill="9" visible="yes" active="yes"/>
 <layer number="146" name="DrillLegend_01-20" color="3" fill="9" visible="yes" active="yes"/>
+<layer number="150" name="Notes" color="7" fill="1" visible="yes" active="yes"/>
 <layer number="151" name="HeatSink" color="7" fill="1" visible="yes" active="yes"/>
 <layer number="152" name="_bDocu" color="7" fill="1" visible="yes" active="yes"/>
+<layer number="153" name="FabDoc1" color="6" fill="1" visible="no" active="no"/>
+<layer number="154" name="FabDoc2" color="2" fill="1" visible="no" active="no"/>
+<layer number="155" name="FabDoc3" color="7" fill="15" visible="no" active="no"/>
 <layer number="199" name="Contour" color="7" fill="1" visible="yes" active="yes"/>
 <layer number="200" name="200bmp" color="7" fill="1" visible="yes" active="yes"/>
@@
 <layer number="225" name="225bmp" color="7" fill="1" visible="yes" active="yes"/>
 <layer number="226" name="226bmp" color="7" fill="1" visible="yes" active="yes"/>
+<layer number="227" name="227bmp" color="7" fill="1" visible="yes" active="yes"/>
+<layer number="228" name="228bmp" color="7" fill="1" visible="yes" active="yes"/>
 <layer number="248" name="Housing" color="7" fill="1" visible="yes" active="yes"/>
 <layer number="249" name="Edge" color="7" fill="1" visible="yes" active="yes"/>
@@
 <wire x1="-0.5" y1="12.5" x2="2.5" y2="15.5" width="1" layer="46" curve="-90"/>
 <wire x1="70.7" y1="15.5" x2="73.7" y2="12.5" width="1" layer="46" curve="-90"/>
-<dimension x1="16.6" y1="-0.5" x2="3.8" y2="-0.5" x3="10.2" y3="-11.7" layer="47" dtype="horizontal"/>
-<dimension x1="16.05" y1="4" x2="4.35" y2="4" x3="10.2" y3="-5.4" layer="47" dtype="horizontal"/>
-<dimension x1="43" y1="-0.5" x2="30.2" y2="-0.5" x3="36.6" y3="-24" layer="47" dtype="horizontal"/>
-<dimension x1="42.45" y1="4" x2="30.75" y2="4" x3="36.6" y3="-18" layer="47" dtype="horizontal"/>
-<dimension x1="69.4" y1="-0.5" x2="56.6" y2="-0.5" x3="63" y3="-11.7" layer="47" dtype="horizontal"/>
-<dimension x1="68.85" y1="4" x2="57.15" y2="4" x3="63" y3="-5.4" layer="47" dtype="horizontal"/>
-<dimension x1="30.2" y1="20" x2="43" y2="20" x3="36.6" y3="31.2" layer="47" dtype="horizontal"/>
-<dimension x1="30.75" y1="15.5" x2="42.45" y2="15.5" x3="36.6" y3="24.9" layer="47" dtype="horizontal"/>
-<dimension x1="0" y1="13.5" x2="73.2" y2="13.55" x3="36.6" y3="39.5" layer="47" dtype="horizontal"/>
-<dimension x1="1.5" y1="15" x2="3.3" y2="0" x3="-18.8" y3="7.5" layer="47" dtype="vertical"/>
-<dimension x1="36.6" y1="-5" x2="16.6" y2="-13.7" x3="26.6" y3="-34.25" layer="47" dtype="horizontal"/>
-<dimension x1="36.6" y1="-2" x2="56.6" y2="-13.7" x3="46.6" y3="-34.25" layer="47" dtype="horizontal"/>
+<dimension x1="16.6" y1="-0.5" x2="3.8" y2="-0.5" x3="10.2" y3="-11.7" textsize="3.5" layer="47" dtype="horizontal"/>
+<dimension x1="16.05" y1="4" x2="4.35" y2="4" x3="10.2" y3="-5.4" textsize="3.5" layer="47" dtype="horizontal"/>
+<dimension x1="43" y1="-0.5" x2="30.2" y2="-0.5" x3="36.6" y3="-24" textsize="3.5" layer="47" dtype="horizontal"/>
+<dimension x1="42.45" y1="4" x2="30.75" y2="4" x3="36.6" y3="-18" textsize="3.5" layer="47" dtype="horizontal"/>
+<dimension x1="69.4" y1="-0.5" x2="56.6" y2="-0.5" x3="63" y3="-11.7" textsize="3.5" layer="47" dtype="horizontal"/>
+<dimension x1="68.85" y1="4" x2="57.15" y2="4" x3="63" y3="-5.4" textsize="3.5" layer="47" dtype="horizontal"/>
+<dimension x1="30.2" y1="20" x2="43" y2="20" x3="36.6" y3="31.2" textsize="3.5" layer="47" dtype="horizontal"/>
+<dimension x1="30.75" y1="15.5" x2="42.45" y2="15.5" x3="36.6" y3="24.9" textsize="3.5" layer="47" dtype="horizontal"/>
+<dimension x1="0" y1="13.5" x2="73.2" y2="13.55" x3="36.6" y3="39.5" textsize="3.5" layer="47" dtype="horizontal"/>
+<dimension x1="1.5" y1="15" x2="3.3" y2="0" x3="-18.8" y3="7.5" textsize="3.5" layer="47" dtype="vertical"/>
+<dimension x1="36.6" y1="-5" x2="16.6" y2="-13.7" x3="26.6" y3="-34.25" textsize="3.5" layer="47" dtype="horizontal"/>
+<dimension x1="36.6" y1="-2" x2="56.6" y2="-13.7" x3="46.6" y3="-34.25" textsize="3.5" layer="47" dtype="horizontal"/>
 <text x="38.05" y="26.65" size="3" layer="47" rot="R90">C.L.</text>
-<dimension x1="3.3" y1="0" x2="-0.5" y2="4.5" x3="-5.6" y3="2.25" layer="47" dtype="vertical"/>
+<dimension x1="3.3" y1="0" x2="-0.5" y2="4.5" x3="-5.6" y3="2.25" textsize="3.5" layer="47" dtype="vertical"/>
 <wire x1="42.95" y1="6.858" x2="42.95" y2="5.842" width="0.1016" layer="145"/>
 <wire x1="42.442" y1="6.35" x2="43.458" y2="6.35" width="0.1016" layer="145"/>
@@
 <wire x1="40.912" y1="17.508" x2="41.42" y2="17.508" width="0.1016" layer="146"/>
 <wire x1="36.6" y1="21.1" x2="36.6" y2="25.95" width="0.1016" layer="47"/>
-<dimension x1="70.7" y1="12.5" x2="73.129253125" y2="13.0905375" x3="80.708521875" y3="14.933009375" layer="47" dtype="radius"/>
-<dimension x1="29.65" y1="19.5" x2="22.85" y2="15" x3="22.85" y3="17.25" layer="47" dtype="vertical"/>
+<dimension x1="70.7" y1="12.5" x2="73.129253125" y2="13.0905375" x3="80.708521875" y3="14.933009375" textsize="3.5" layer="47" dtype="radius"/>
+<dimension x1="29.65" y1="19.5" x2="22.85" y2="15" x3="22.85" y3="17.25" textsize="3.5" layer="47" dtype="vertical"/>
 <text x="20.7" y="48.75" size="1.778" layer="46">1mm DIA. ROUTER PATH</text>
-<dimension x1="16.6" y1="3.5" x2="30.2" y2="3.5" x3="23.4" y3="5.25" layer="47"/>
+<dimension x1="16.6" y1="3.5" x2="30.2" y2="3.5" x3="23.4" y3="5.25" textsize="3.5" layer="47"/>
 <text x="68.45" y="12.15" size="1.778" layer="21" font="vector" rot="SR270">fork</text>
 <text x="70.65" y="11.3" size="1.778" layer="21" font="vector" rot="SR270">w7</text>
@@
 </class>
 </classes>
-<designrules>
+<designrules name="default">
 <description language="en">&lt;b&gt;EAGLE Design Rules&lt;/b&gt;
 &lt;p&gt;
@@
 <element name="W7BSF3" library="bitSnap" package="BITSNAP_V03_FEMALE" value="BITSNAP_V03_FEMALE" x="56.55" y="0"/>
 <element name="W7BSM1" library="bitSnap" package="BITSNAP_V03_MALE" value="BITSNAP_V03_MALE" x="43.05" y="19.5" rot="R180"/>
-<element name="FRAME1" library="LITTLEBITS" package="FABDWG01-OHW" value="FRAME-LETTER-OHWOHW" x="-128.46" y="-81.4"/>
-<element name="U$12" library="LITTLEBITS" package="OSHWCREDIT" value="OSHWCREDIT" x="-39.1" y="-79.35"/>
-<element name="U$1" library="LITTLEBITS" package="OSHW-LOGO-L" value="" x="-6.95" y="-75.65"/>
+<element name="FRAME1" library="LITTLEBITS" package="FABDWG01-OHW" value="FRAME-LETTER-OHWOHW" x="28.44" y="-5.85"/>
+<element name="U$12" library="LITTLEBITS" package="OSHWCREDIT" value="OSHWCREDIT" x="-63.75" y="-71.75"/>
+<element name="U$2" library="LITTLEBITS" package="OSHW-LOGO-L" value="OSHW-LOGOL" x="-9.45" y="-66.55"/>
 </elements>
 <signals>
@@
 </board>
 </drawing>
+<compatibility>
+<note version="6.3" minversion="6.2.2" severity="warning">
+Since Version 6.2.2 text objects can contain more than one line,
+which will not be processed correctly with this version.
+</note>
+</compatibility>
 </eagle>

Commit message: Updated license text
Parts:
- moved U$2 10.6 mm to (-4.45, -75.9)
Changed lines of the file:
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@@
 <element name="FRAME1" library="LITTLEBITS" package="FABDWG01-OHW" value="FRAME-LETTER-OHWOHW" x="28.44" y="-5.85"/>
 <element name="U$12" library="LITTLEBITS" package="OSHWCREDIT" value="OSHWCREDIT" x="-63.75" y="-71.75"/>
-<element name="U$2" library="LITTLEBITS" package="OSHW-LOGO-L" value="OSHW-LOGOL" x="-9.45" y="-66.55"/>
+<element name="U$2" library="LITTLEBITS" package="OSHW-LOGO-L" value="OSHW-LOGOL" x="-4.45" y="-75.9"/>
 </elements>
 <signals>
