File: WIRE/LB_BIT_w8-LATCH/LB_BIT_w8-latch_v03(1_1)/LB_BIT_w8-latch_v03(1_1).brd (EAGLE design)
At the start: 21.4 x 11.5 mm, 17 parts

Commit message: Updated license text
Parts:
- moved U$2 5.10 mm to (-91.7, -62.6)
Changed lines of the file:
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@@
 <?xml version="1.0" encoding="utf-8"?>
 <!DOCTYPE eagle SYSTEM "eagle.dtd">
-<eagle version="6.5.0">
+<eagle version="6.6.0">
 <drawing>
 <settings>
@@
 <attribute name="LB_PN" value="?" x="17.1" y="9.76" size="1.778" layer="27" rot="R90" display="off"/>
 <attribute name="V_OPERATION" value="5V" x="17.1" y="9.76" size="1.778" layer="27" rot="R90" display="off"/>
-<attribute name="IEC_ESD_PROT" value="+/-18kV" x="17.1" y="9.76" size="1.778" layer="27" rot="R90" display="off"/>
 <attribute name="V_CLAMP" value="?" x="17.1" y="9.76" size="1.778" layer="27" rot="R90" display="off"/>
 <attribute name="NAME" x="18.016" y="10.929" size="0.4064" layer="25" rot="R270"/>
 <attribute name="VALUE" x="19.097" y="7.844" size="0.4064" layer="27" rot="R90"/>
+<attribute name="MPN" value="ESD9B5.0ST5G" x="17.1" y="9.76" size="1.778" layer="27" rot="R90" display="off"/>
+<attribute name="IEC_ESD_PROT0" value="+/-18kV" x="17.1" y="9.76" size="1.778" layer="27" rot="R90" display="off"/>
 </element>
 <element name="W8R3" library="SparkFun" package="0603-RES" value="1K" x="12" y="10.56" smashed="yes">
@@
 </element>
 <element name="U$1" library="LITTLEBITS" package="OSHW-LOGO-L" value="OSHW-LOGOL" x="-24.65" y="-71.1"/>
-<element name="U$2" library="LITTLEBITS" package="OSHWCREDIT" value="OSHWCREDIT" x="-94.1" y="-67.1"/>
+<element name="U$2" library="LITTLEBITS" package="OSHWCREDIT" value="OSHWCREDIT" x="-91.7" y="-62.6"/>
 <element name="U$12" library="LITTLEBITS" package="FABDWG01-OHW" value="FRAME-LETTER-OHWOHW" x="0" y="0"/>
 </elements>
