File: INPUT/LB_BIT_i30_KEYBOARD/LB_BIT_i30_KEYBOARD-v03(3_4)/LB_BIT_i30_KEYBOARD-v03(3_4)-OHW.brd (EAGLE design)
At the start: 21.4 x 84.1 mm, 55 parts

Commit message: Updated licenses
Parts:
- moved U$2 13.2 mm to (-15.6, -66.3)
Changed lines of the file:
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@@
 <?xml version="1.0" encoding="utf-8"?>
 <!DOCTYPE eagle SYSTEM "eagle.dtd">
-<eagle version="6.4">
+<eagle version="6.6.0">
 <drawing>
 <settings>
@@
 <layer number="225" name="225bmp" color="26" fill="10" visible="yes" active="yes"/>
 <layer number="226" name="226bmp" color="27" fill="10" visible="yes" active="yes"/>
+<layer number="227" name="227bmp" color="7" fill="1" visible="yes" active="yes"/>
+<layer number="228" name="228bmp" color="7" fill="1" visible="yes" active="yes"/>
 <layer number="248" name="Housing" color="7" fill="1" visible="yes" active="yes"/>
 <layer number="249" name="Edge" color="7" fill="1" visible="yes" active="yes"/>
@@
 <attribute name="VALUE" x="-7.903" y="1.666" size="0.4064" layer="28" rot="MR270"/>
 </element>
-<element name="U$2" library="LITTLEBITS" package="OSHWCREDIT-KORG" value="OSHWCREDIT-KORG" x="-2.4" y="-67.45"/>
+<element name="U$2" library="LITTLEBITS" package="OSHWCREDIT-KORG" value="OSHWCREDIT-KORG" x="-15.55" y="-66.35"/>
 </elements>
 <signals>

Commit message: Updated license text
Parts:
- moved U$2 9.71 mm to (-25.2, -65.8)
Changed lines of the file:
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@@
 <attribute name="VALUE" x="-7.903" y="1.666" size="0.4064" layer="28" rot="MR270"/>
 </element>
-<element name="U$2" library="LITTLEBITS" package="OSHWCREDIT-KORG" value="OSHWCREDIT-KORG" x="-15.55" y="-66.35"/>
+<element name="U$2" library="LITTLEBITS" package="OSHWCREDIT-KORG" value="OSHWCREDIT-KORG" x="-25.25" y="-65.85"/>
 </elements>
 <signals>

Commit message: Updated license in Korg bits modules
Parts:
- moved U$2 2.75 mm to (-27.9, -65.1)
Changed lines of the file:
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@@
 <layer number="111" name="LB_TEXT" color="13" fill="1" visible="yes" active="yes"/>
 <layer number="112" name="tSilk" color="7" fill="1" visible="yes" active="yes"/>
+<layer number="113" name="ReferenceLS" color="7" fill="1" visible="yes" active="yes"/>
 <layer number="116" name="Patch_BOT" color="9" fill="4" visible="yes" active="yes"/>
+<layer number="118" name="Rect_Pads" color="7" fill="1" visible="yes" active="yes"/>
 <layer number="121" name="_tsilk" color="7" fill="1" visible="yes" active="yes"/>
 <layer number="122" name="_bsilk" color="7" fill="1" visible="yes" active="yes"/>
@@
 <attribute name="VALUE" x="-7.903" y="1.666" size="0.4064" layer="28" rot="MR270"/>
 </element>
-<element name="U$2" library="LITTLEBITS" package="OSHWCREDIT-KORG" value="OSHWCREDIT-KORG" x="-25.25" y="-65.85"/>
+<element name="U$2" library="LITTLEBITS" package="OSHWCREDIT-KORG" value="OSHWCREDIT-KORG" x="-27.9" y="-65.1"/>
 </elements>
 <signals>
