File: INPUT/LB_BIT_i33_ENVELOPE/LB_BIT_i33_envelope-v03(3_3).brd (EAGLE design)
At the start: 21.4 x 37.9 mm, 66 parts

Commit message: Updated licenses
Parts:
- removed U$7: OSHWCREDIT-KORG, LITTLEBITS:OSHWCREDIT-KORG
- added U$3: OSHWCREDIT-KORG, LITTLEBITS:OSHWCREDIT-KORG
- renumbered FRAME1 to U$1
Changed lines of the file:
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@@
 <?xml version="1.0" encoding="utf-8"?>
 <!DOCTYPE eagle SYSTEM "eagle.dtd">
-<eagle version="6.4">
+<eagle version="6.6.0">
 <drawing>
 <settings>
@@
 <layer number="225" name="225bmp" color="26" fill="10" visible="yes" active="yes"/>
 <layer number="226" name="226bmp" color="27" fill="10" visible="yes" active="yes"/>
+<layer number="227" name="227bmp" color="7" fill="1" visible="yes" active="yes"/>
+<layer number="228" name="228bmp" color="7" fill="1" visible="yes" active="yes"/>
 <layer number="248" name="Housing" color="7" fill="1" visible="yes" active="yes"/>
 <layer number="249" name="Edge" color="7" fill="1" visible="yes" active="yes"/>
@@
 <attribute name="VALUE" x="-44.507" y="38.066" size="0.4064" layer="28" font="vector" rot="MR270"/>
 </element>
-<element name="FRAME1" library="LITTLEBITS" package="FABDWG01-OHW" value="FRAME-LETTER-OHWOHW" x="0" y="0" locked="yes"/>
 <element name="I33C8" library="LITTLEBITS" package="CAP-0603" value="0.1uF" x="-52.95" y="36.5" smashed="yes" rot="MR90">
 <attribute name="LB_PN" value="" x="-52.95" y="36.5" size="1.778" layer="28" rot="MR90" display="off"/>
@@
 <attribute name="VOLTAGE" value="" x="-41.6" y="37.1" size="1.778" layer="28" rot="MR0" display="off"/>
 </element>
-<element name="U$7" library="LITTLEBITS" package="OSHWCREDIT-KORG" value="OSHWCREDIT-KORG" x="-53.75" y="-75.1"/>
 <element name="U$9" library="LITTLEBITS" package="OSHW-LOGO-L" value="OSHW-LOGOL" x="-23.85" y="-71.15"/>
+<element name="U$1" library="LITTLEBITS" package="FABDWG01-OHW" value="FRAME-LETTER-OHWOHW" x="0" y="0"/>
+<element name="U$3" library="LITTLEBITS" package="OSHWCREDIT-KORG" value="OSHWCREDIT-KORG" x="-61.3" y="-77.3"/>
 </elements>
 <signals>

Commit message: Updated license in Korg bits modules
Parts:
- moved U$3 17.7 mm to (-76.7, -68.6)
- moved U$9 7.82 mm to (-29.5, -65.8)
Changed lines of the file:
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@@
 <layer number="111" name="LB_TEXT" color="13" fill="1" visible="yes" active="yes"/>
 <layer number="112" name="tSilk" color="7" fill="1" visible="yes" active="yes"/>
+<layer number="113" name="ReferenceLS" color="7" fill="1" visible="yes" active="yes"/>
 <layer number="116" name="Patch_BOT" color="9" fill="4" visible="yes" active="yes"/>
+<layer number="118" name="Rect_Pads" color="7" fill="1" visible="yes" active="yes"/>
 <layer number="121" name="_tsilk" color="7" fill="1" visible="yes" active="yes"/>
 <layer number="122" name="_bsilk" color="7" fill="1" visible="yes" active="yes"/>
@@
 <attribute name="VOLTAGE" value="" x="-41.6" y="37.1" size="1.778" layer="28" rot="MR0" display="off"/>
 </element>
-<element name="U$9" library="LITTLEBITS" package="OSHW-LOGO-L" value="OSHW-LOGOL" x="-23.85" y="-71.15"/>
+<element name="U$9" library="LITTLEBITS" package="OSHW-LOGO-L" value="OSHW-LOGOL" x="-29.5" y="-65.75"/>
 <element name="U$1" library="LITTLEBITS" package="FABDWG01-OHW" value="FRAME-LETTER-OHWOHW" x="0" y="0"/>
-<element name="U$3" library="LITTLEBITS" package="OSHWCREDIT-KORG" value="OSHWCREDIT-KORG" x="-61.3" y="-77.3"/>
+<element name="U$3" library="LITTLEBITS" package="OSHWCREDIT-KORG" value="OSHWCREDIT-KORG" x="-76.7" y="-68.6"/>
 </elements>
 <signals>
