File: INPUT/LB_BIT_i37_MIX/LB_BIT_i37_mix_in-v03(1_1)/LB_BIT_i37_mix_in-v03(1_1).brd (EAGLE design)
At the start: 21.4 x 9.4 mm, 6 parts

Commit message: Updated licenses
Parts:
- moved U$4 8.07 mm to (-61.0, -78.2)
- renumbered FRAME1 to U$1
Changed lines of the file:
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@@
 <?xml version="1.0" encoding="utf-8"?>
 <!DOCTYPE eagle SYSTEM "eagle.dtd">
-<eagle version="6.4">
+<eagle version="6.6.0">
 <drawing>
 <settings>
@@
 <layer number="225" name="225bmp" color="26" fill="10" visible="yes" active="yes"/>
 <layer number="226" name="226bmp" color="27" fill="10" visible="yes" active="yes"/>
+<layer number="227" name="227bmp" color="7" fill="1" visible="yes" active="yes"/>
+<layer number="228" name="228bmp" color="7" fill="1" visible="yes" active="yes"/>
 <layer number="248" name="Housing" color="7" fill="1" visible="yes" active="yes"/>
 <layer number="249" name="Edge" color="7" fill="1" visible="yes" active="yes"/>
@@
 <element name="U$3" library="SparkFun" package="OSHW-LOGO-L" value="OSHW-LOGOL" x="-25.34" y="-72.09"/>
 <element name="U$2" library="ohw-logo" package="OSHW_FILLX150_NOTEXT" value="" x="15.789" y="2.629"/>
-<element name="U$4" library="LITTLEBITS" package="OSHWCREDIT-KORG" value="OSHWCREDIT-KORG" x="-53.43" y="-75.58"/>
 <element name="I37BSF1" library="bitSnap" package="BITSNAP_V03_MALE" value="BITSNAP_V03_MALE" x="16.65" y="12.95" rot="R180"/>
-<element name="FRAME1" library="LITTLEBITS" package="FABDWG01-OHW" value="FRAME-LETTER-OHWOHW" x="0" y="0" locked="yes"/>
+<element name="U$1" library="LITTLEBITS" package="FABDWG01-OHW" value="FRAME-LETTER-OHWOHW" x="0" y="0"/>
+<element name="U$4" library="LITTLEBITS" package="OSHWCREDIT-KORG" value="OSHWCREDIT-KORG" x="-61.05" y="-78.25"/>
 </elements>
 <signals>

Commit message: Updated license in Korg bits modules
Parts:
- moved U$4 17.4 mm to (-77.3, -72.2)
Changed lines of the file:
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@@
 <layer number="111" name="LB_TEXT" color="13" fill="1" visible="yes" active="yes"/>
 <layer number="112" name="tSilk" color="7" fill="1" visible="yes" active="yes"/>
+<layer number="113" name="ReferenceLS" color="7" fill="1" visible="yes" active="yes"/>
 <layer number="116" name="Patch_BOT" color="9" fill="4" visible="yes" active="yes"/>
+<layer number="118" name="Rect_Pads" color="7" fill="1" visible="yes" active="yes"/>
 <layer number="121" name="_tsilk" color="7" fill="1" visible="yes" active="yes"/>
 <layer number="122" name="_bsilk" color="7" fill="1" visible="yes" active="yes"/>
@@
 <element name="I37BSF1" library="bitSnap" package="BITSNAP_V03_MALE" value="BITSNAP_V03_MALE" x="16.65" y="12.95" rot="R180"/>
 <element name="U$1" library="LITTLEBITS" package="FABDWG01-OHW" value="FRAME-LETTER-OHWOHW" x="0" y="0"/>
-<element name="U$4" library="LITTLEBITS" package="OSHWCREDIT-KORG" value="OSHWCREDIT-KORG" x="-61.05" y="-78.25"/>
+<element name="U$4" library="LITTLEBITS" package="OSHWCREDIT-KORG" value="OSHWCREDIT-KORG" x="-77.35" y="-72.25"/>
 </elements>
 <signals>
