File: OUTPUT/LB_BIT_o24_SYNTHSPEAKER/LB_BIT_o24_SYNTHSPEAKER-v03(4_5)/LB_BIT_o24_SYNTHSPEAKER-v03(4_5).brd (EAGLE design)
At the start: 27.2 x 51.1 mm, 31 parts

Commit message: Updated licenses
Parts:
- removed $1_27_$: OSHWCREDIT-KORG, LITTLEBITS:OSHWCREDIT-KORG
- added U$1: OSHWCREDIT-KORG, LITTLEBITS:OSHWCREDIT-KORG

Commit message: Updated license in Korg bits modules
Parts:
- moved U$1 18.0 mm to (-24.5, -55.6)
- moved $1_28_$ 2.75 mm to (24.4, -52.2)
Changed lines of the file:
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@@
 <layer number="111" name="LB_TEXT" color="13" fill="1" visible="yes" active="yes"/>
 <layer number="112" name="tSilk" color="7" fill="1" visible="yes" active="yes"/>
+<layer number="113" name="ReferenceLS" color="7" fill="1" visible="yes" active="yes"/>
 <layer number="116" name="Patch_BOT" color="9" fill="4" visible="yes" active="yes"/>
+<layer number="118" name="Rect_Pads" color="7" fill="1" visible="yes" active="yes"/>
 <layer number="121" name="_tsilk" color="7" fill="1" visible="yes" active="yes"/>
 <layer number="122" name="_bsilk" color="7" fill="1" visible="yes" active="yes"/>
@@
 <attribute name="VALUE" x="11.707" y="22.534" size="0.4064" layer="28" font="vector" rot="MR0"/>
 </element>
-<element name="$1_28_$" library="LITTLEBITS" package="OSHW-LOGO-L" value="OSHW-LOGOL" x="24.45" y="-55"/>
+<element name="$1_28_$" library="LITTLEBITS" package="OSHW-LOGO-L" value="OSHW-LOGOL" x="24.45" y="-52.25"/>
 <element name="O24C6" library="LITTLEBITS" package="CAP-0603" value="0.1uF" x="9.2" y="23.85" smashed="yes" rot="MR270">
 <attribute name="LB_PN" value="" x="9.2" y="23.85" size="1.778" layer="28" rot="MR270" display="off"/>
@@
 <attribute name="VOLTAGE" value="" x="10.4" y="44.45" size="1.778" layer="28" rot="MR90" display="off"/>
 </element>
-<element name="U$1" library="LITTLEBITS" package="OSHWCREDIT-KORG" value="OSHWCREDIT-KORG" x="-8.3" y="-63.6"/>
+<element name="U$1" library="LITTLEBITS" package="OSHWCREDIT-KORG" value="OSHWCREDIT-KORG" x="-24.5" y="-55.65"/>
 </elements>
 <signals>
