File: WIRE/LB_BIT_w19_SPLIT/LB_w19_SPLIT_IN/LB_w19_SPLIT_IN-v03(rev2_2)/LB_w19_SPLIT_IN-v03(rev2_2)-OHW.sch (EAGLE design)
At the start: 11 parts

Commit message: Updated license in Korg bits modules
Changed lines of the file:
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@@
 <?xml version="1.0" encoding="utf-8"?>
 <!DOCTYPE eagle SYSTEM "eagle.dtd">
-<eagle version="6.5.0">
+<eagle version="6.6.0">
 <drawing>
 <settings>
@@
 <layer number="111" name="LB_TEXT" color="13" fill="1" visible="yes" active="yes"/>
 <layer number="112" name="tSilk" color="7" fill="1" visible="yes" active="yes"/>
+<layer number="113" name="ReferenceLS" color="7" fill="1" visible="yes" active="yes"/>
 <layer number="116" name="Patch_BOT" color="9" fill="4" visible="yes" active="yes"/>
+<layer number="118" name="Rect_Pads" color="7" fill="1" visible="yes" active="yes"/>
 <layer number="121" name="_tsilk" color="7" fill="1" visible="yes" active="yes"/>
 <layer number="122" name="_bsilk" color="7" fill="1" visible="yes" active="yes"/>
@@
 <layer number="225" name="225bmp" color="26" fill="10" visible="no" active="yes"/>
 <layer number="226" name="226bmp" color="27" fill="10" visible="no" active="yes"/>
+<layer number="227" name="227bmp" color="7" fill="1" visible="yes" active="yes"/>
+<layer number="228" name="228bmp" color="7" fill="1" visible="yes" active="yes"/>
 <layer number="248" name="Housing" color="7" fill="1" visible="yes" active="yes"/>
 <layer number="249" name="Edge" color="7" fill="1" visible="yes" active="yes"/>
@@
 <instance part="W19JP1" gate="G$1" x="185.42" y="114.3" rot="MR0"/>
 <instance part="U$3" gate="G$1" x="134.62" y="10.16"/>
-<instance part="U$4" gate="G$1" x="43.18" y="12.7"/>
+<instance part="U$4" gate="G$1" x="33.02" y="12.7"/>
 <instance part="W19BSM1" gate="G$1" x="101.6" y="104.14"/>
 <instance part="W19JP2" gate="G$1" x="185.42" y="93.98" rot="MR0"/>
