File: WIRE/LB_w19_SPLIT/LB_w19_SPLIT_OUT/LB_w19_SPLIT_OUT-v03(rev1_1)/LB_w19_SPLIT_OUT-v03(rev1_1).brd (EAGLE design)
At the start: 21.4 x 9.4 mm, 6 parts

Commit message: Updated license in Korg bits modules
Parts:
- moved U$1 15.7 mm to (-77.3, -71.5)
Changed lines of the file:
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@@
 <layer number="111" name="LB_TEXT" color="13" fill="1" visible="yes" active="yes"/>
 <layer number="112" name="tSilk" color="7" fill="1" visible="yes" active="yes"/>
+<layer number="113" name="ReferenceLS" color="7" fill="1" visible="yes" active="yes"/>
 <layer number="116" name="Patch_BOT" color="9" fill="4" visible="yes" active="yes"/>
+<layer number="118" name="Rect_Pads" color="7" fill="1" visible="yes" active="yes"/>
 <layer number="121" name="_tsilk" color="7" fill="1" visible="yes" active="yes"/>
 <layer number="122" name="_bsilk" color="7" fill="1" visible="yes" active="yes"/>
@@
 <element name="W19BSF1" library="bitSnap" package="BITSNAP_V03_FEMALE" value="BITSNAP_V03_FEMALE" x="3.75" y="0"/>
 <element name="FRAME1" library="LITTLEBITS" package="FABDWG01-OHW" value="FRAME-LETTER-OHWOHW" x="0" y="0"/>
-<element name="U$1" library="LITTLEBITS" package="OSHWCREDIT-KORG" value="OSHWCREDIT-KORG" x="-61.95" y="-74.4"/>
+<element name="U$1" library="LITTLEBITS" package="OSHWCREDIT-KORG" value="OSHWCREDIT-KORG" x="-77.35" y="-71.5"/>
 </elements>
 <signals>
